File: Mainboard.sch (KiCad schematic (older format))
At the start: 34 parts

Commit message: Add files via upload
Parts:
- added BZ?: Buzzer, symbol Device:Buzzer
- added D?: CABLE_DETECT, symbol Device:LED
- added R? (x2): 10k, symbol Device:R_Small
- added R? (x3): 470, symbol Device:R_Small
Connections:
- net labels added: VDD
- wire segments 153 -> 165
Changed lines of the file:
@@
 L power:GND #PWR?
 U 1 1 5DB9DB5B
-P 5200 7600
-F 0 "#PWR?" H 5200 7350 50  0001 C CNN
-F 1 "GND" H 5205 7427 50  0000 C CNN
-F 2 "" H 5200 7600 50  0001 C CNN
-F 3 "" H 5200 7600 50  0001 C CNN
-	1    5200 7600
-	1    0    0    -1
-$EndComp
-Wire Wire Line
-	5200 7600 5200 7350
+P 4700 7600
+F 0 "#PWR?" H 4700 7350 50  0001 C CNN
+F 1 "GND" H 4705 7427 50  0000 C CNN
+F 2 "" H 4700 7600 50  0001 C CNN
+F 3 "" H 4700 7600 50  0001 C CNN
+	1    4700 7600
+	1    0    0    -1
+$EndComp
+Wire Wire Line
+	4700 7600 4700 7350
 Wire Wire Line
 	5200 7350 5450 7350
@@
 F1 "power.sch" 50
 $EndSheet
+$Comp
+L Device:Buzzer BZ?
+U 1 1 5DBF25B1
+P 7650 4550
+F 0 "BZ?" H 7802 4579 50  0000 L CNN
+F 1 "Buzzer" H 7802 4488 50  0000 L CNN
+F 2 "" V 7625 4650 50  0001 C CNN
+F 3 "~" V 7625 4650 50  0001 C CNN
+	1    7650 4550
+	1    0    0    -1
+$EndComp
+Wire Wire Line
+	5650 2750 5450 2750
+$Comp
+L Device:R_Small R?
+U 1 1 5DC08487
+P 5250 2650
+F 0 "R?" V 5446 2650 50  0000 C CNN
+F 1 "10k" V 5355 2650 50  0000 C CNN
+F 2 "" H 5250 2650 50  0001 C CNN
+F 3 "~" H 5250 2650 50  0001 C CNN
+	1    5250 2650
+	0    -1   -1   0
+$EndComp
+$Comp
+L Device:R_Small R?
+U 1 1 5DC08F93
+P 5250 2850
+F 0 "R?" V 5446 2850 50  0000 C CNN
+F 1 "10k" V 5355 2850 50  0000 C CNN
+F 2 "" H 5250 2850 50  0001 C CNN
+F 3 "~" H 5250 2850 50  0001 C CNN
+	1    5250 2850
+	0    -1   -1   0
+$EndComp
+Wire Wire Line
+	5450 2750 5450 2650
+Wire Wire Line
+	5450 2650 5350 2650
+Wire Wire Line
+	5450 2750 5450 2850
+Wire Wire Line
+	5450 2850 5350 2850
+Connection ~ 5450 2750
+$Comp
+L power:GND #PWR?
+U 1 1 5DC615DF
+P 5050 2900
+F 0 "#PWR?" H 5050 2650 50  0001 C CNN
+F 1 "GND" H 5055 2727 50  0000 C CNN
+F 2 "" H 5050 2900 50  0001 C CNN
+F 3 "" H 5050 2900 50  0001 C CNN
+	1    5050 2900
+	1    0    0    -1
+$EndComp
+Wire Wire Line
+	5050 2900 5050 2850
+Wire Wire Line
+	5050 2850 5150 2850
+Wire Wire Line
+	5050 2650 5150 2650
+$Comp
+L power:VDD #PWR?
+U 1 1 5DC7CCF8
+P 5050 2650
+F 0 "#PWR?" H 5050 2500 50  0001 C CNN
+F 1 "VDD" H 5067 2823 50  0000 C CNN
+F 2 "" H 5050 2650 50  0001 C CNN
+F 3 "" H 5050 2650 50  0001 C CNN
+	1    5050 2650
+	1    0    0    -1
+$EndComp
+Wire Wire Line
+	6850 4450 7550 4450
+$Comp
+L power:GND #PWR?
+U 1 1 5DC8DCD7
+P 7550 4750
+F 0 "#PWR?" H 7550 4500 50  0001 C CNN
+F 1 "GND" H 7555 4577 50  0000 C CNN
+F 2 "" H 7550 4750 50  0001 C CNN
+F 3 "" H 7550 4750 50  0001 C CNN
+	1    7550 4750
+	1    0    0    -1
+$EndComp
+Wire Wire Line
+	7550 4750 7550 4650
+$Comp
+L Device:R_Small R?
+U 1 1 5DCA6D89
+P 5100 7350
+F 0 "R?" V 4904 7350 50  0000 C CNN
+F 1 "470" V 4995 7350 50  0000 C CNN
+F 2 "" H 5100 7350 50  0001 C CNN
+F 3 "~" H 5100 7350 50  0001 C CNN
+	1    5100 7350
+	0    1    1    0
+$EndComp
+$Comp
+L Device:LED D?
+U 1 1 5DCA786C
+P 4850 7350
+F 0 "D?" H 4843 7566 50  0000 C CNN
+F 1 "CABLE_DETECT" H 4843 7475 50  0000 C CNN
+F 2 "" H 4850 7350 50  0001 C CNN
+F 3 "~" H 4850 7350 50  0001 C CNN
+	1    4850 7350
+	1    0    0    -1
+$EndComp
+Wire Wire Line
+	6250 6850 6550 6850
+Wire Wire Line
+	6250 7450 6550 7450
+Text Label 6550 6850 2    50   ~ 0
+CAN_RX
+Text Label 6550 7450 2    50   ~ 0
+CAN_TX
+$Comp
+L Device:R_Small R?
+U 1 1 5DCF3973
+P 6250 7250
+F 0 "R?" H 6309 7296 50  0000 L CNN
+F 1 "470" H 6309 7205 50  0000 L CNN
+F 2 "" H 6250 7250 50  0001 C CNN
+F 3 "~" H 6250 7250 50  0001 C CNN
+	1    6250 7250
+	1    0    0    -1
+$EndComp
+$Comp
+L Device:R_Small R?
+U 1 1 5DCF45CE
+P 6250 6650
+F 0 "R?" H 6309 6696 50  0000 L CNN
+F 1 "470" H 6309 6605 50  0000 L CNN
+F 2 "" H 6250 6650 50  0001 C CNN
+F 3 "~" H 6250 6650 50  0001 C CNN
+	1    6250 6650
+	1    0    0    -1
+$EndComp
+$Comp
+L power:+3.3V #PWR?
+U 1 1 5DCF51EA
+P 6250 6550
+F 0 "#PWR?" H 6250 6400 50  0001 C CNN
+F 1 "+3.3V" H 6265 6723 50  0000 C CNN
+F 2 "" H 6250 6550 50  0001 C CNN
+F 3 "" H 6250 6550 50  0001 C CNN
+	1    6250 6550
+	1    0    0    -1
+$EndComp
+$Comp
+L power:+3.3V #PWR?
+U 1 1 5DCF594A
+P 6250 7150
+F 0 "#PWR?" H 6250 7000 50  0001 C CNN
+F 1 "+3.3V" H 6265 7323 50  0000 C CNN
+F 2 "" H 6250 7150 50  0001 C CNN
+F 3 "" H 6250 7150 50  0001 C CNN
+	1    6250 7150
+	1    0    0    -1
+$EndComp
 $EndSCHEMATC

Commit message: Add files via upload
Connections:
- net labels removed: MISO1, MOSI1, SCLK1
- wire segments 165 -> 162
Changed lines of the file:
@@
 SCL
 Wire Wire Line
-	6850 3450 7200 3450
-Wire Wire Line
-	6850 3350 7200 3350
-Wire Wire Line
-	6850 3250 7200 3250
-Wire Wire Line
-	6850 3150 7200 3150
-Text Label 7200 3350 2    50   ~ 0
-SCLK1
-Text Label 7200 3250 2    50   ~ 0
-MOSI1
-Text Label 7200 3150 2    50   ~ 0
-MISO1
+	6850 4350 7200 4350
 $Comp
 L power:GND #PWR?
@@
 Text Label 9050 6100 0    50   ~ 0
 MAG_CS
-Text Label 7200 3450 2    50   ~ 0
+Text Label 7200 4350 2    50   ~ 0
 IMU_CS
 Text Label 7200 4850 2    50   ~ 0
 MAG_CS
-Text Label 9050 5700 0    50   ~ 0
-MISO1
-Text Label 9050 5800 0    50   ~ 0
-MOSI1
-Text Label 9050 5900 0    50   ~ 0
-SCLK1
 Text Label 7200 4150 2    50   ~ 0
 MOSI
@@
 	1    0    0    -1
 $EndComp
+Text Label 9050 5700 0    50   ~ 0
+MISO
+Text Label 9050 5800 0    50   ~ 0
+MOSI
+Text Label 9050 5900 0    50   ~ 0
+SCLK
 $EndSCHEMATC

Commit message: Added flash chip
Parts:
- added R? (x2): 10k, symbol Device:R
- added U?: W25N01GV, symbol iclr:W25N01GV
Connections:
- wire segments 162 -> 177
Changed lines of the file:
@@
 EESchema Schematic File Version 4
 LIBS:Mainboard-cache
-EELAYER 30 0
+EELAYER 29 0
 EELAYER END
 $Descr A4 11693 8268
@@
 Text Label 9050 5900 0    50   ~ 0
 SCLK
+$Comp
+L iclr:W25N01GV U?
+U 1 1 5DBDFA30
+P 7950 5850
+F 0 "U?" H 7950 6300 50  0000 C CNN
+F 1 "W25N01GV" H 7950 6200 50  0000 C CNN
+F 2 "" H 7950 5850 50  0001 C CNN
+F 3 "" H 7950 5850 50  0001 C CNN
+	1    7950 5850
+	1    0    0    -1
+$EndComp
+$Comp
+L power:+3.3V #PWR?
+U 1 1 5DBE112C
+P 8350 5350
+F 0 "#PWR?" H 8350 5200 50  0001 C CNN
+F 1 "+3.3V" H 8400 5550 50  0000 C CNN
+F 2 "" H 8350 5350 50  0001 C CNN
+F 3 "" H 8350 5350 50  0001 C CNN
+	1    8350 5350
+	1    0    0    -1
+$EndComp
+Wire Wire Line
+	8300 5700 8350 5700
+Wire Wire Line
+	8350 5700 8350 5400
+$Comp
+L power:GND #PWR?
+U 1 1 5DBE9FD9
+P 7950 6300
+F 0 "#PWR?" H 7950 6050 50  0001 C CNN
+F 1 "GND" H 8000 6100 50  0000 C CNN
+F 2 "" H 7950 6300 50  0001 C CNN
+F 3 "" H 7950 6300 50  0001 C CNN
+	1    7950 6300
+	1    0    0    -1
+$EndComp
+Wire Wire Line
+	7950 6300 7950 6250
+Wire Wire Line
+	7600 6000 7550 6000
+Wire Wire Line
+	7550 6000 7550 6250
+Wire Wire Line
+	7550 6250 7950 6250
+Connection ~ 7950 6250
+Wire Wire Line
+	7950 6250 7950 6200
+$Comp
+L Device:R R?
+U 1 1 5DBFB89C
+P 8600 5600
+F 0 "R?" H 8700 5650 50  0000 L CNN
+F 1 "10k" H 8700 5600 50  0000 L CNN
+F 2 "" V 8530 5600 50  0001 C CNN
+F 3 "~" H 8600 5600 50  0001 C CNN
+	1    8600 5600
+	1    0    0    -1
+$EndComp
+Wire Wire Line
+	8300 5800 8600 5800
+Wire Wire Line
+	8600 5800 8600 5750
+Wire Wire Line
+	8350 5400 8600 5400
+Wire Wire Line
+	8600 5400 8600 5450
+Connection ~ 8350 5400
+Wire Wire Line
+	8350 5400 8350 5350
+$Comp
+L Device:R R?
+U 1 1 5DC1F150
+P 7300 5700
+F 0 "R?" H 7200 5650 50  0000 R CNN
+F 1 "10k" H 7200 5700 50  0000 R CNN
+F 2 "" V 7230 5700 50  0001 C CNN
+F 3 "~" H 7300 5700 50  0001 C CNN
+	1    7300 5700
+	1    0    0    1
+$EndComp
+Wire Wire Line
+	7300 5850 7300 5900
+Wire Wire Line
+	7300 5900 7600 5900
+$Comp
+L power:+3.3V #PWR?
+U 1 1 5DC42464
+P 7300 5350
+F 0 "#PWR?" H 7300 5200 50  0001 C CNN
+F 1 "+3.3V" H 7350 5550 50  0000 C CNN
+F 2 "" H 7300 5350 50  0001 C CNN
+F 3 "" H 7300 5350 50  0001 C CNN
+	1    7300 5350
+	1    0    0    -1
+$EndComp
+Wire Wire Line
+	7300 5350 7300 5550
 $EndSCHEMATC

Commit message: Add files via upload
Connections:
- wire segments 177 -> 181
Other:
- moved on the sheet: R?
Changed lines of the file:
@@
 EESchema Schematic File Version 4
 LIBS:Mainboard-cache
-EELAYER 29 0
+EELAYER 30 0
 EELAYER END
 $Descr A4 11693 8268
@@
 L iclr:W25N01GV U?
 U 1 1 5DBDFA30
-P 7950 5850
-F 0 "U?" H 7950 6300 50  0000 C CNN
-F 1 "W25N01GV" H 7950 6200 50  0000 C CNN
-F 2 "" H 7950 5850 50  0001 C CNN
-F 3 "" H 7950 5850 50  0001 C CNN
-	1    7950 5850
+P 7600 1400
+F 0 "U?" H 7600 1850 50  0000 C CNN
+F 1 "W25N01GV" H 7600 1750 50  0000 C CNN
+F 2 "" H 7600 1400 50  0001 C CNN
+F 3 "" H 7600 1400 50  0001 C CNN
+	1    7600 1400
 	1    0    0    -1
 $EndComp
@@
 L power:+3.3V #PWR?
 U 1 1 5DBE112C
-P 8350 5350
-F 0 "#PWR?" H 8350 5200 50  0001 C CNN
-F 1 "+3.3V" H 8400 5550 50  0000 C CNN
-F 2 "" H 8350 5350 50  0001 C CNN
-F 3 "" H 8350 5350 50  0001 C CNN
-	1    8350 5350
-	1    0    0    -1
-$EndComp
-Wire Wire Line
-	8300 5700 8350 5700
-Wire Wire Line
-	8350 5700 8350 5400
+P 8000 900
+F 0 "#PWR?" H 8000 750 50  0001 C CNN
+F 1 "+3.3V" H 8050 1100 50  0000 C CNN
+F 2 "" H 8000 900 50  0001 C CNN
+F 3 "" H 8000 900 50  0001 C CNN
+	1    8000 900
+	1    0    0    -1
+$EndComp
+Wire Wire Line
+	7950 1250 8000 1250
+Wire Wire Line
+	8000 1250 8000 950
 $Comp
 L power:GND #PWR?
 U 1 1 5DBE9FD9
-P 7950 6300
-F 0 "#PWR?" H 7950 6050 50  0001 C CNN
-F 1 "GND" H 8000 6100 50  0000 C CNN
-F 2 "" H 7950 6300 50  0001 C CNN
-F 3 "" H 7950 6300 50  0001 C CNN
-	1    7950 6300
-	1    0    0    -1
-$EndComp
-Wire Wire Line
-	7950 6300 7950 6250
-Wire Wire Line
-	7600 6000 7550 6000
-Wire Wire Line
-	7550 6000 7550 6250
-Wire Wire Line
-	7550 6250 7950 6250
-Connection ~ 7950 6250
-Wire Wire Line
-	7950 6250 7950 6200
+P 7600 1850
+F 0 "#PWR?" H 7600 1600 50  0001 C CNN
+F 1 "GND" H 7650 1650 50  0000 C CNN
+F 2 "" H 7600 1850 50  0001 C CNN
+F 3 "" H 7600 1850 50  0001 C CNN
+	1    7600 1850
+	1    0    0    -1
+$EndComp
+Wire Wire Line
+	7600 1850 7600 1800
+Wire Wire Line
+	7250 1550 7200 1550
+Wire Wire Line
+	7200 1550 7200 1800
+Wire Wire Line
+	7200 1800 7600 1800
+Connection ~ 7600 1800
+Wire Wire Line
+	7600 1800 7600 1750
 $Comp
 L Device:R R?
 U 1 1 5DBFB89C
-P 8600 5600
-F 0 "R?" H 8700 5650 50  0000 L CNN
-F 1 "10k" H 8700 5600 50  0000 L CNN
-F 2 "" V 8530 5600 50  0001 C CNN
-F 3 "~" H 8600 5600 50  0001 C CNN
-	1    8600 5600
-	1    0    0    -1
-$EndComp
-Wire Wire Line
-	8300 5800 8600 5800
-Wire Wire Line
-	8600 5800 8600 5750
-Wire Wire Line
-	8350 5400 8600 5400
-Wire Wire Line
-	8600 5400 8600 5450
-Connection ~ 8350 5400
-Wire Wire Line
-	8350 5400 8350 5350
+P 8250 1150
+F 0 "R?" H 8350 1200 50  0000 L CNN
+F 1 "10k" H 8350 1150 50  0000 L CNN
+F 2 "" V 8180 1150 50  0001 C CNN
+F 3 "~" H 8250 1150 50  0001 C CNN
+	1    8250 1150
+	1    0    0    -1
+$EndComp
+Wire Wire Line
+	7950 1350 8250 1350
+Wire Wire Line
+	8250 1350 8250 1300
+Wire Wire Line
+	8000 950  8250 950
+Wire Wire Line
+	8250 950  8250 1000
+Connection ~ 8000 950
+Wire Wire Line
+	8000 950  8000 900
 $Comp
 L Device:R R?
 U 1 1 5DC1F150
-P 7300 5700
-F 0 "R?" H 7200 5650 50  0000 R CNN
-F 1 "10k" H 7200 5700 50  0000 R CNN
-F 2 "" V 7230 5700 50  0001 C CNN
-F 3 "~" H 7300 5700 50  0001 C CNN
-	1    7300 5700
+P 6800 1250
+F 0 "R?" H 6700 1200 50  0000 R CNN
+F 1 "10k" H 6700 1250 50  0000 R CNN
+F 2 "" V 6730 1250 50  0001 C CNN
+F 3 "~" H 6800 1250 50  0001 C CNN
+	1    6800 1250
 	1    0    0    1
 $EndComp
 Wire Wire Line
-	7300 5850 7300 5900
-Wire Wire Line
-	7300 5900 7600 5900
+	6800 1400 6800 1450
 $Comp
 L power:+3.3V #PWR?
 U 1 1 5DC42464
-P 7300 5350
-F 0 "#PWR?" H 7300 5200 50  0001 C CNN
-F 1 "+3.3V" H 7350 5550 50  0000 C CNN
-F 2 "" H 7300 5350 50  0001 C CNN
-F 3 "" H 7300 5350 50  0001 C CNN
-	1    7300 5350
-	1    0    0    -1
-$EndComp
-Wire Wire Line
-	7300 5350 7300 5550
+P 6800 900
+F 0 "#PWR?" H 6800 750 50  0001 C CNN
+F 1 "+3.3V" H 6850 1100 50  0000 C CNN
+F 2 "" H 6800 900 50  0001 C CNN
+F 3 "" H 6800 900 50  0001 C CNN
+	1    6800 900
+	1    0    0    -1
+$EndComp
+Wire Wire Line
+	6800 900  6800 1100
+Wire Wire Line
+	7950 1550 8250 1550
+Wire Wire Line
+	7950 1450 8250 1450
+Wire Wire Line
+	6800 1450 7250 1450
+Wire Wire Line
+	7250 1350 6950 1350
+Wire Wire Line
+	7250 1250 6950 1250
+Text Label 8250 1450 2    50   ~ 0
+SCLK
+Text Label 8250 1550 2    50   ~ 0
+MOSI
+Text Label 6950 1350 0    50   ~ 0
+MISO
+Text Label 6950 1250 0    50   ~ 0
+FLASH_CS
 $EndSCHEMATC

Commit message: Add files via upload
Parts:
- removed JP?: XBEE, XBEE, symbol Sparkfun_RF:XBEE
- added JP?: XBEE, XBEE, symbol iclr:XBEE
Changed lines of the file:
@@
 RADIO_TX
-$Comp
-L Sparkfun_RF:XBEE JP?
-U 1 1 5DB6F306
-P 10350 3150
-F 0 "JP?" H 10350 3910 45  0000 C CNN
-F 1 "XBEE" H 10350 3826 45  0000 C CNN
-F 2 "XBEE" H 10350 3750 20  0001 C CNN
-F 3 "" H 10350 3150 50  0001 C CNN
-F 4 "XXX-00000" H 10350 3731 60  0000 C CNN "Field4"
-	1    10350 3150
-	1    0    0    -1
-$EndComp
 $Comp
 L power:GND #PWR?
@@
 Text Label 6950 1250 0    50   ~ 0
 FLASH_CS
+$Comp
+L iclr:XBEE JP?
+U 1 1 5DBE2F9A
+P 10350 3150
+F 0 "JP?" H 10350 3910 45  0000 C CNN
+F 1 "XBEE" H 10350 3826 45  0000 C CNN
+F 2 "XBEE" H 10350 3750 20  0001 C CNN
+F 3 "" H 10350 3150 50  0001 C CNN
+F 4 "XXX-00000" H 10350 3731 60  0000 C CNN "Field4"
+	1    10350 3150
+	1    0    0    -1
+$EndComp
 $EndSCHEMATC

Commit message: Add files via upload
Parts:
- gave numbers to parts that had none: 44
Connections:
- wire segments 181 -> 184
Other:
- moved on the sheet: D5, R13

Commit message: installed the nukes
Connections:
- net labels added: Cont1, Cont2, Nuke1, Nuke2
- wire segments 184 -> 192
Other:
- moved on the sheet: BZ1
Changed lines of the file:
@@
 $Descr A4 11693 8268
 encoding utf-8
-Sheet 1 4
+Sheet 1 5
 Title ""
 Date ""
@@
 L Device:Buzzer BZ1
 U 1 1 5DBF25B1
-P 7650 4550
-F 0 "BZ1" H 7802 4579 50  0000 L CNN
-F 1 "Buzzer" H 7802 4488 50  0000 L CNN
-F 2 "" V 7625 4650 50  0001 C CNN
-F 3 "~" V 7625 4650 50  0001 C CNN
-	1    7650 4550
+P 8100 4550
+F 0 "BZ1" H 8252 4579 50  0000 L CNN
+F 1 "Buzzer" H 8252 4488 50  0000 L CNN
+F 2 "" V 8075 4650 50  0001 C CNN
+F 3 "~" V 8075 4650 50  0001 C CNN
+	1    8100 4550
 	1    0    0    -1
 $EndComp
@@
 L power:GND #PWR0129
 U 1 1 5DC8DCD7
-P 7550 4750
-F 0 "#PWR0129" H 7550 4500 50  0001 C CNN
-F 1 "GND" H 7555 4577 50  0000 C CNN
-F 2 "" H 7550 4750 50  0001 C CNN
-F 3 "" H 7550 4750 50  0001 C CNN
-	1    7550 4750
-	1    0    0    -1
-$EndComp
-Wire Wire Line
-	7550 4750 7550 4650
+P 8000 4750
+F 0 "#PWR0129" H 8000 4500 50  0001 C CNN
+F 1 "GND" H 8005 4577 50  0000 C CNN
+F 2 "" H 8000 4750 50  0001 C CNN
+F 3 "" H 8000 4750 50  0001 C CNN
+	1    8000 4750
+	1    0    0    -1
+$EndComp
+Wire Wire Line
+	8000 4750 8000 4650
 $Comp
 L Device:R_Small R13
@@
 Wire Wire Line
 	5350 7350 5450 7350
+$Sheet
+S 7800 5600 800  500
+U 5DDE1103
+F0 "nukes" 50
+F1 "Nukes.sch" 50
+F2 "Nuke1" I L 7800 5700 50
+F3 "Cont1" I L 7800 5800 50
+F4 "Nuke2" I L 7800 5900 50
+F5 "Cont2" I L 7800 6000 50
+$EndSheet
+Wire Wire Line
+	6850 3150 7200 3150
+Wire Wire Line
+	6850 3250 7200 3250
+Wire Wire Line
+	6850 3350 7200 3350
+Wire Wire Line
+	6850 3450 7200 3450
+Text Label 7200 3150 2    50   ~ 0
+Nuke1
+Text Label 7200 3250 2    50   ~ 0
+Cont1
+Text Label 7200 3350 2    50   ~ 0
+Nuke2
+Text Label 7200 3450 2    50   ~ 0
+Cont2
+Wire Wire Line
+	7800 5700 7450 5700
+Wire Wire Line
+	7800 5800 7450 5800
+Wire Wire Line
+	7800 5900 7450 5900
+Wire Wire Line
+	7800 6000 7450 6000
+Text Label 7450 5700 0    50   ~ 0
+Nuke1
+Text Label 7450 5800 0    50   ~ 0
+Cont1
+Text Label 7450 5900 0    50   ~ 0
+Nuke2
+Text Label 7450 6000 0    50   ~ 0
+Cont2
 $EndSCHEMATC

Commit message: Add files via upload
Parts:
- added D?: D_Schottky, Diode_SMD:D_SOD-123F, symbol Device:D_Schottky
- added Q?: PMV20ENR, Package_TO_SOT_SMD:SOT-23, symbol Device:Q_NMOS_GSD
Connections:
- wire segments 192 -> 194
Other:
- moved on the sheet: BZ1
Changed lines of the file:
@@
 L Device:Buzzer BZ1
 U 1 1 5DBF25B1
-P 8100 4550
-F 0 "BZ1" H 8252 4579 50  0000 L CNN
-F 1 "Buzzer" H 8252 4488 50  0000 L CNN
-F 2 "" V 8075 4650 50  0001 C CNN
-F 3 "~" V 8075 4650 50  0001 C CNN
-	1    8100 4550
+P 8150 3650
+F 0 "BZ1" H 8302 3679 50  0000 L CNN
+F 1 "Buzzer" H 8302 3588 50  0000 L CNN
+F 2 "" V 8125 3750 50  0001 C CNN
+F 3 "~" V 8125 3750 50  0001 C CNN
+	1    8150 3650
 	1    0    0    -1
 $EndComp
@@
 	1    0    0    -1
 $EndComp
-Wire Wire Line
-	6850 4450 7550 4450
-$Comp
-L power:GND #PWR0129
-U 1 1 5DC8DCD7
-P 8000 4750
-F 0 "#PWR0129" H 8000 4500 50  0001 C CNN
-F 1 "GND" H 8005 4577 50  0000 C CNN
-F 2 "" H 8000 4750 50  0001 C CNN
-F 3 "" H 8000 4750 50  0001 C CNN
-	1    8000 4750
-	1    0    0    -1
-$EndComp
-Wire Wire Line
-	8000 4750 8000 4650
 $Comp
 L Device:R_Small R13
@@
 Text Label 7450 6000 0    50   ~ 0
 Cont2
+$Comp
+L Device:Q_NMOS_GSD Q?
+U 1 1 5DE0D306
+P 7950 4450
+AR Path="/5DDE6CFA/5DE0D306" Ref="Q?"  Part="1"
+AR Path="/5DDE1103/5DE0D306" Ref="Q?"  Part="1"
+AR Path="/5DE0D306" Ref="Q?"  Part="1"
+F 0 "Q?" H 8156 4496 50  0000 L CNN
+F 1 "PMV20ENR" H 8156 4405 50  0000 L CNN
+F 2 "Package_TO_SOT_SMD:SOT-23" H 8150 4550 50  0001 C CNN
+F 3 "~" H 7950 4450 50  0001 C CNN
+	1    7950 4450
+	1    0    0    -1
+$EndComp
+$Comp
+L power:GND #PWR?
+U 1 1 5DE0D30D
+P 8050 4900
+AR Path="/5DDE6CFA/5DE0D30D" Ref="#PWR?"  Part="1"
+AR Path="/5DDE1103/5DE0D30D" Ref="#PWR?"  Part="1"
+AR Path="/5DE0D30D" Ref="#PWR?"  Part="1"
+F 0 "#PWR?" H 8050 4650 50  0001 C CNN
+F 1 "GND" H 8055 4727 50  0000 C CNN
+F 2 "" H 8050 4900 50  0001 C CNN
+F 3 "" H 8050 4900 50  0001 C CNN
+	1    8050 4900
+	1    0    0    -1
+$EndComp
+$Comp
+L Device:D_Schottky D?
+U 1 1 5DE49A6B
+P 8050 4000
+AR Path="/5DAD2180/5DE49A6B" Ref="D?"  Part="1"
+AR Path="/5DB4FA2A/5DE49A6B" Ref="D?"  Part="1"
+AR Path="/5DDE6CFA/5DE49A6B" Ref="D?"  Part="1"
+AR Path="/5DDE1103/5DE49A6B" Ref="D?"  Part="1"
+AR Path="/5DE49A6B" Ref="D?"  Part="1"
+F 0 "D?" V 8096 3921 50  0000 R CNN
+F 1 "D_Schottky" V 8005 3921 50  0000 R CNN
+F 2 "Diode_SMD:D_SOD-123F" H 8050 4000 50  0001 C CNN
+F 3 "http://www.smc-diodes.com/propdf/DSS12U%20THRU%20DSS125U%20N1873%20REV.A.pdf" H 8050 4000 50  0001 C CNN
+	1    8050 4000
+	0    -1   -1   0
+$EndComp
+Wire Wire Line
+	8050 4150 8050 4250
+Wire Wire Line
+	8050 3750 8050 3850
+Wire Wire Line
+	8050 4650 8050 4900
+Wire Wire Line
+	6850 4450 7750 4450
+$Comp
+L power:+3.3V #PWR?
+U 1 1 5DEC6485
+P 8050 3550
+F 0 "#PWR?" H 8050 3400 50  0001 C CNN
+F 1 "+3.3V" H 8065 3723 50  0000 C CNN
+F 2 "" H 8050 3550 50  0001 C CNN
+F 3 "" H 8050 3550 50  0001 C CNN
+	1    8050 3550
+	1    0    0    -1
+$EndComp
 $EndSCHEMATC
