File: IMU.sch (KiCad schematic (older format))
At the start: 0 parts

Commit message: update IMU
Parts:
- added C? (x3): 100nF, symbol Device:C_Small
- added C?: 10uF, symbol Device:C_Small
- added C?: 10nF, symbol Device:C_Small
- added U?: LSM9DS1, Package_LGA:LGA-24L_3x3.5mm_P0.43mm, symbol Sensor_Motion:LSM9DS1
Connections:
- net labels added: +3.3V, GND, SDO_M
- wire segments 0 -> 35
