File: IMU.sch (KiCad schematic (older format))
At the start: 6 parts

Commit message: Add files via upload
Parts:
- C5, C6, C7, C8, C9: renamed from C?; footprint (none) -> Capacitor_SMD:C_0603_1608Metric
- gave numbers to parts that had none: 1
Changed lines of the file:
@@
 $Descr A4 11693 8268
 encoding utf-8
-Sheet 3 4
+Sheet 3 5
 Title ""
 Date ""
@@
 MAG_CS
 $Comp
-L Sensor_Motion:LSM9DS1 U?
+L Sensor_Motion:LSM9DS1 U7
 U 1 1 5DBB7353
 P 6750 2500
-F 0 "U?" H 6750 1611 50  0000 C CNN
+F 0 "U7" H 6750 1611 50  0000 C CNN
 F 1 "LSM9DS1" H 6750 1520 50  0000 C CNN
 F 2 "Package_LGA:LGA-24L_3x3.5mm_P0.43mm" H 8250 3250 50  0001 C CNN
@@
 Connection ~ 7450 2600
 $Comp
-L power:GND #PWR?
+L power:GND #PWR048
 U 1 1 5DBBA85D
 P 7600 2600
-F 0 "#PWR?" H 7600 2350 50  0001 C CNN
+F 0 "#PWR048" H 7600 2350 50  0001 C CNN
 F 1 "GND" V 7605 2472 50  0000 R CNN
 F 2 "" H 7600 2600 50  0001 C CNN
@@
 P 6800 1400
 AR Path="/5DBC6E2A" Ref="C?"  Part="1"
-AR Path="/5DBB30BF/5DBC6E2A" Ref="C?"  Part="1"
-F 0 "C?" V 6571 1400 50  0000 C CNN
+AR Path="/5DBB30BF/5DBC6E2A" Ref="C8"  Part="1"
+F 0 "C8" V 6571 1400 50  0000 C CNN
 F 1 "100nF" V 6662 1400 50  0000 C CNN
-F 2 "" H 6800 1400 50  0001 C CNN
+F 2 "Capacitor_SMD:C_0603_1608Metric" H 6800 1400 50  0001 C CNN
 F 3 "~" H 6800 1400 50  0001 C CNN
 	1    6800 1400
@@
 P 7150 1400
 AR Path="/5DBC8962" Ref="C?"  Part="1"
-AR Path="/5DBB30BF/5DBC8962" Ref="C?"  Part="1"
-F 0 "C?" V 6921 1400 50  0000 C CNN
+AR Path="/5DBB30BF/5DBC8962" Ref="C9"  Part="1"
+F 0 "C9" V 6921 1400 50  0000 C CNN
 F 1 "10uF" V 7012 1400 50  0000 C CNN
-F 2 "" H 7150 1400 50  0001 C CNN
+F 2 "Capacitor_SMD:C_0603_1608Metric" H 7150 1400 50  0001 C CNN
 F 3 "~" H 7150 1400 50  0001 C CNN
 	1    7150 1400
@@
 	7250 1600 7500 1600
 $Comp
-L power:GND #PWR?
+L power:GND #PWR046
 U 1 1 5DBC9BD7
 P 7150 1300
-F 0 "#PWR?" H 7150 1050 50  0001 C CNN
+F 0 "#PWR046" H 7150 1050 50  0001 C CNN
 F 1 "GND" H 7155 1127 50  0000 C CNN
 F 2 "" H 7150 1300 50  0001 C CNN
@@
 $EndComp
 $Comp
-L power:GND #PWR?
+L power:GND #PWR045
 U 1 1 5DBCA3AF
 P 6800 1300
-F 0 "#PWR?" H 6800 1050 50  0001 C CNN
+F 0 "#PWR045" H 6800 1050 50  0001 C CNN
 F 1 "GND" H 6805 1127 50  0000 C CNN
 F 2 "" H 6800 1300 50  0001 C CNN
@@
 $EndComp
 $Comp
-L power:+3.3V #PWR?
+L power:+3.3V #PWR047
 U 1 1 5DBCADD4
 P 7500 1450
-F 0 "#PWR?" H 7500 1300 50  0001 C CNN
+F 0 "#PWR047" H 7500 1300 50  0001 C CNN
 F 1 "+3.3V" H 7515 1623 50  0000 C CNN
 F 2 "" H 7500 1450 50  0001 C CNN
@@
 	6750 1700 6350 1700
 $Comp
-L power:+3.3V #PWR?
+L power:+3.3V #PWR044
 U 1 1 5DBCC221
 P 6550 1500
-F 0 "#PWR?" H 6550 1350 50  0001 C CNN
+F 0 "#PWR044" H 6550 1350 50  0001 C CNN
 F 1 "+3.3V" H 6565 1673 50  0000 C CNN
 F 2 "" H 6550 1500 50  0001 C CNN
@@
 P 6250 1400
 AR Path="/5DBCCB7B" Ref="C?"  Part="1"
-AR Path="/5DBB30BF/5DBCCB7B" Ref="C?"  Part="1"
-F 0 "C?" V 6021 1400 50  0000 C CNN
+AR Path="/5DBB30BF/5DBCCB7B" Ref="C7"  Part="1"
+F 0 "C7" V 6021 1400 50  0000 C CNN
 F 1 "100nF" V 6112 1400 50  0000 C CNN
-F 2 "" H 6250 1400 50  0001 C CNN
+F 2 "Capacitor_SMD:C_0603_1608Metric" H 6250 1400 50  0001 C CNN
 F 3 "~" H 6250 1400 50  0001 C CNN
 	1    6250 1400
@@
 $EndComp
 $Comp
-L power:GND #PWR?
+L power:GND #PWR043
 U 1 1 5DBCCF0A
 P 6250 1300
-F 0 "#PWR?" H 6250 1050 50  0001 C CNN
+F 0 "#PWR043" H 6250 1050 50  0001 C CNN
 F 1 "GND" H 6255 1127 50  0000 C CNN
 F 2 "" H 6250 1300 50  0001 C CNN
@@
 P 5800 3600
 AR Path="/5DBD5269" Ref="C?"  Part="1"
-AR Path="/5DBB30BF/5DBD5269" Ref="C?"  Part="1"
-F 0 "C?" V 5571 3600 50  0000 C CNN
+AR Path="/5DBB30BF/5DBD5269" Ref="C6"  Part="1"
+F 0 "C6" V 5571 3600 50  0000 C CNN
 F 1 "100nF" V 5662 3600 50  0000 C CNN
-F 2 "" H 5800 3600 50  0001 C CNN
+F 2 "Capacitor_SMD:C_0603_1608Metric" H 5800 3600 50  0001 C CNN
 F 3 "~" H 5800 3600 50  0001 C CNN
 	1    5800 3600
@@
 P 5800 3250
 AR Path="/5DBD639A" Ref="C?"  Part="1"
-AR Path="/5DBB30BF/5DBD639A" Ref="C?"  Part="1"
-F 0 "C?" V 5571 3250 50  0000 C CNN
+AR Path="/5DBB30BF/5DBD639A" Ref="C5"  Part="1"
+F 0 "C5" V 5571 3250 50  0000 C CNN
 F 1 "10nF" V 5662 3250 50  0000 C CNN
-F 2 "" H 5800 3250 50  0001 C CNN
+F 2 "Capacitor_SMD:C_0603_1608Metric" H 5800 3250 50  0001 C CNN
 F 3 "~" H 5800 3250 50  0001 C CNN
 	1    5800 3250
@@
 	5900 3000 5900 3250
 $Comp
-L power:GND #PWR?
+L power:GND #PWR042
 U 1 1 5DBD8595
 P 5700 3600
-F 0 "#PWR?" H 5700 3350 50  0001 C CNN
+F 0 "#PWR042" H 5700 3350 50  0001 C CNN
 F 1 "GND" V 5705 3472 50  0000 R CNN
 F 2 "" H 5700 3600 50  0001 C CNN
@@
 $EndComp
 $Comp
-L power:GND #PWR?
+L power:GND #PWR041
 U 1 1 5DBD8EEE
 P 5700 3250
-F 0 "#PWR?" H 5700 3000 50  0001 C CNN
+F 0 "#PWR041" H 5700 3000 50  0001 C CNN
 F 1 "GND" V 5705 3122 50  0000 R CNN
 F 2 "" H 5700 3250 50  0001 C CNN

Commit message: Add files via upload
Connections:
- wire segments 35 -> 37
Changed lines of the file:
@@
 Text HLabel 5800 2100 0    50   Input ~ 0
 SCLK
-Text HLabel 4800 2800 0    50   Input ~ 0
+Text HLabel 5800 2400 0    50   Input ~ 0
 IMU_CS
-Text HLabel 4800 2950 0    50   Input ~ 0
+Text HLabel 7750 2100 2    50   Input ~ 0
 MAG_CS
 $Comp
@@
 Wire Wire Line
 	5800 2200 6050 2200
+Wire Wire Line
+	7750 2100 7450 2100
+Wire Wire Line
+	6050 2400 5800 2400
 $EndSCHEMATC

Commit message: Add files via upload
Connections:
- no-connect marks 0 -> 5
