File: Nukes.sch (KiCad schematic (older format))
At the start: 14 parts

Commit message: installed the nukes
Parts:
- removed D? (x2): DIODE, Diode_SMD:D_SMA, symbol Device:D
- removed D? (x2): FIRING, LED_SMD:LED_0805_2012Metric, symbol Device:LED
- removed J? (x4): Screw_Terminal_01x02, TerminalBlock_Phoenix:TerminalBlock_Phoenix_MPT-0,5-2-2.54_1x02_P2.54mm_Horizontal, symbol Connector:Screw_Terminal_01x02
- removed JP? (x2): SolderJumper_3_Open, Jumper:SolderJumper-3_P2.0mm_Open_TrianglePad1.0x1.5mm, symbol Jumper:SolderJumper_3_Open
- removed Q? (x2): Q_NMOS_GSD, Package_TO_SOT_SMD:SOT-23, symbol Device:Q_NMOS_GSD
- removed R? (x2): 1k, Resistor_SMD:R_0603_1608Metric, symbol Device:R
- added D? (x2): FIRING, LED_SMD:LED_0603_1608Metric_Castellated, symbol Device:LED
- added D? (x2): D_Schottky, Diode_SMD:D_SOD-123F, symbol Device:D_Schottky
- added D? (x2): CONTINUITY, LED_SMD:LED_0603_1608Metric_Castellated, symbol Device:LED
- added D? (x2): ARM, LED_SMD:LED_0603_1608Metric_Castellated, symbol Device:LED
- added J? (x4): Screw_Terminal_01x02, TerminalBlock_Phoenix:TerminalBlock_Phoenix_MPT-0,5-2-2.54_1x02_P2.54mm_Horizontal, symbol Connector:Screw_Terminal_01x02
- added JP? (x2): SolderJumper_3_Open, Jumper:SolderJumper-3_P1.3mm_Open_RoundedPad1.0x1.5mm_NumberLabels, symbol Jumper:SolderJumper_3_Open
- added Q? (x2): PMV20ENR, Package_TO_SOT_SMD:SOT-23, symbol Device:Q_NMOS_GSD
- added R? (x6): 470, Resistor_SMD:R_0603_1608Metric, symbol Device:R
- added R? (x4): 500, Resistor_SMD:R_0603_1608Metric, symbol Device:R
- added SW? (x2): SW_DPDT_x2, Button_Switch_THT:SW_CuK_JS202011AQN_DPDT_Angled, symbol Switch:SW_DPDT_x2
- added SW? (x2): SW_DPDT_x2, symbol Switch:SW_DPDT_x2
- added U? (x2): LTV-817S, Package_DIP:SMDIP-4_W9.53mm, symbol Isolator:LTV-817S
Connections:
- net labels added: CONT, Cont1, Cont2, Nuke1, Nuke2
- wire segments 124 -> 178
Other:
- note added: "External ematch supply"
- note removed: "External ematch supply\n"
