File: Nukes.sch (KiCad schematic (older format))
At the start: 21 parts, among them J6 Screw_Terminal_01x02, J7 Screw_Terminal_01x02, J8 Screw_Terminal_01x02, Q4 PMV20ENR, Q5 PMV20ENR, U10 LTV-817S, U9 LTV-817S

Commit message: update
Parts:
- R27, R30, R32, R35: value 1k -> 1K
Changed lines of the file:
@@
 AR Path="/5DDE1103/5DE04B01" Ref="R32"  Part="1"
 F 0 "R32" H 7920 4496 50  0000 L CNN
-F 1 "1k" H 7920 4405 50  0000 L CNN
+F 1 "1K" H 7920 4405 50  0000 L CNN
 F 2 "Resistor_SMD:R_0603_1608Metric" V 7780 4450 50  0001 C CNN
 F 3 "~" H 7850 4450 50  0001 C CNN
@@
 AR Path="/5DDE1103/5DE04B5E" Ref="R35"  Part="1"
 F 0 "R35" H 10220 4696 50  0000 L CNN
-F 1 "1k" H 10220 4605 50  0000 L CNN
+F 1 "1K" H 10220 4605 50  0000 L CNN
 F 2 "Resistor_SMD:R_0603_1608Metric" V 10080 4650 50  0001 C CNN
 F 3 "~" H 10150 4650 50  0001 C CNN
@@
 AR Path="/5DDE1103/5DE3233E" Ref="R27"  Part="1"
 F 0 "R27" H 3620 4646 50  0000 L CNN
-F 1 "1k" H 3620 4555 50  0000 L CNN
+F 1 "1K" H 3620 4555 50  0000 L CNN
 F 2 "Resistor_SMD:R_0603_1608Metric" V 3480 4600 50  0001 C CNN
 F 3 "~" H 3550 4600 50  0001 C CNN
@@
 AR Path="/5DDE1103/5DE3239B" Ref="R30"  Part="1"
 F 0 "R30" H 5970 4846 50  0000 L CNN
-F 1 "1k" H 5970 4755 50  0000 L CNN
+F 1 "1K" H 5970 4755 50  0000 L CNN
 F 2 "Resistor_SMD:R_0603_1608Metric" V 5830 4800 50  0001 C CNN
 F 3 "~" H 5900 4800 50  0001 C CNN
