File: Mainboard.kicad_pcb (KiCad board)
At the start: 2 copper layers, 135 parts, among them J1 USB_B_Micro, J10 Conn_01x02_Male, J11 Conn_01x02_Male, J12 Conn_01x02_Male, J2 8P8C_LED, J3 Micro_SD_Card_Det, J4 Conn_Coaxial, J5 Conn_Coaxial, J6 Screw_Terminal_01x02, J7 Screw_Terminal_01x02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

Commit message: REEEEEEEEE
Parts:
- moved TP23 369.4 mm to (533.5, 83.7)
- moved C12 345.9 mm to (526.4, 142.3)
- moved C13 341.8 mm to (526.4, 140.8)
- moved TP19 339.4 mm to (536.5, 83.9)
- moved U4 302.3 mm to (460.0, -6.00)
- moved TP24 299.0 mm to (458.0, -17.0)
- moved C14 298.9 mm to (476.8, 175.7)
- moved R20 298.0 mm to (453.0, -6.00)
- moved JP4 297.8 mm to (538.0, 13.0)
- moved C7 296.9 mm to (539.0, 90.3), turned to 270 degrees
- moved U10 295.3 mm to (538.0, -1.00)
- moved JP5 294.9 mm to (462.0, -12.0)
- moved C15 294.8 mm to (476.8, 174.2)
- moved U7 294.5 mm to (533.9, 89.7), turned to 180 degrees
- moved U9 294.1 mm to (538.0, 7.00)
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Connections:
- J1 pad 2: Net-(D1-Pad4) -> Net-(D1-Pad3)
- J1 pad 3: Net-(D1-Pad3) -> Net-(D1-Pad4)
- U1 pad 3: Net-(D1-Pad3) -> Net-(D1-Pad4)
- U1 pad 4: Net-(D1-Pad4) -> Net-(D1-Pad3)
Routing:
- added copper zone on In2.Cu, net +3V3
- added copper zone on In1.Cu, net GND
Other:
- board outline added: 100 x 60 mm
- copper layers 2 -> 4

Commit message: boneless
Parts:
- added REF**: MountingHole_3.2mm_M3_DIN965_Pad, MountingHole:MountingHole_3.2mm_M3_DIN965_Pad, F.Cu at (182.0, 53.1)
- added REF**: MountingHole_3.2mm_M3_DIN965_Pad, MountingHole:MountingHole_3.2mm_M3_DIN965_Pad, F.Cu at (181.9, 107.0)
- added REF**: MountingHole_3.2mm_M3_DIN965_Pad, MountingHole:MountingHole_3.2mm_M3_DIN965_Pad, F.Cu at (88.0, 53.1)
- added REF**: MountingHole_3.2mm_M3_DIN965_Pad, MountingHole:MountingHole_3.2mm_M3_DIN965_Pad, F.Cu at (88.1, 106.9)
- moved TP19 395.6 mm to (141.0, 74.0)
- moved C7 394.7 mm to (144.6, 78.7)
- moved TP23 394.6 mm to (139.1, 74.0)
- moved C6 394.2 mm to (142.9, 82.4)
- moved U7 394.1 mm to (139.9, 78.4)
- moved C5 392.8 mm to (141.4, 82.4)
- moved R35 392.7 mm to (161.5, 86.0), turned to 90 degrees
- moved C9 391.5 mm to (139.9, 82.4)
- moved C8 390.1 mm to (138.5, 82.4)
- moved C20 389.1 mm to (87.0, 78.2), turned to 180 degrees
- moved C21 388.3 mm to (87.0, 79.7), turned to 180 degrees
- moved Q4 387.3 mm to (162.4, 97.4), turned to 270 degrees
- moved D16 384.4 mm to (161.5, 89.3), turned to 270 degrees
- moved U9 381.6 mm to (165.3, 89.0), turned to 90 degrees
- moved D11 380.8 mm to (162.8, 100.3)
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
Commit message: Add files via upload
Parts:
- moved JP4 3.23 mm to (174.4, 98.6)
- moved C5 2.98 mm to (138.5, 82.8)
- moved R6 2.60 mm to (109.7, 94.9), turned to 0 degrees
- moved JP3 1.83 mm to (177.0, 98.6)
- moved C9 1.54 mm to (141.4, 82.8)
- moved C8 1.54 mm to (139.9, 82.8)
- moved C23 1.11 mm to (114.1, 94.7)
- moved C22 1.11 mm to (115.6, 94.7)
- moved Q1 0.74 mm to (108.7, 92.0), turned to 180 degrees
- moved U1 0.63 mm to (110.9, 98.8)
- moved C6 0.46 mm to (142.9, 82.8)
Routing:
- net +3V3: track 0.00 -> 86.4 mm
- net GND: track 0.00 -> 47.7 mm
- net /CAN_RX: track 0.00 -> 39.0 mm
- net Net-(JP5-Pad2): track 0.00 -> 37.0 mm
- net Net-(D1-Pad2): track 0.00 -> 34.4 mm
- net /CAN_HIGH: track 0.00 -> 28.5 mm
- net /CAN_LOW: track 0.00 -> 20.0 mm
- net /CAN_TX: track 0.00 -> 19.2 mm
- net VDD: track 0.00 -> 17.0 mm
- net Net-(J4-Pad1): track 0.00 -> 15.9 mm
- net Net-(D1-Pad3): track 0.00 -> 15.9 mm
- net Net-(R3-Pad2): track 0.00 -> 15.1 mm
- net Net-(D1-Pad4): track 0.00 -> 13.9 mm
- net Net-(D14-Pad2): track 0.00 -> 13.7 mm
- net Net-(R23-Pad2): track 0.00 -> 11.6 mm
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Other:
- net class thin added: clearance 0.2, trace_width 0.2, via_dia 0.8, via_drill 0.4

Commit message: Add files via upload
Routing:
- net /MOSI: track 11.1 -> 144.9 mm, vias 0 -> 6
- net /SCLK: track 7.38 -> 124.8 mm, vias 0 -> 8
- net /MISO: track 7.66 -> 122.4 mm, vias 0 -> 6
- net /SD_CS: track 3.57 -> 108.4 mm
- net /LORA_INT: track 0.00 -> 92.5 mm, vias 0 -> 2
- net /LORA_RESET: track 0.00 -> 89.4 mm, vias 0 -> 2
- net Net-(R16-Pad2): track 1.45 -> 76.3 mm, vias 0 -> 2
- net /RXD: track 5.88 -> 75.9 mm, vias 0 -> 2
- net /TXD: track 5.87 -> 73.7 mm, vias 0 -> 2
- net /CAN_TX: track 19.2 -> 67.1 mm
- net /RADIO_RX: track 10.6 -> 48.2 mm, vias 0 -> 1
- net /RADIO_TX: track 6.90 -> 44.2 mm
- net /DTR: track 4.29 -> 38.1 mm, vias 0 -> 2
- net Net-(JP5-Pad2): track 37.0 -> 5.22 mm
- net /RTS: track 10.6 -> 40.9 mm, vias 0 -> 2
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
Commit message: pcb update
Parts:
- moved R23 3.98 mm to (157.3, 70.0)
Routing:
- net /SCL: track 8.66 -> 112.1 mm, vias 0 -> 2
- net /SDA: track 5.22 -> 104.8 mm, vias 0 -> 2
- net /BOOT: track 7.82 -> 82.7 mm, vias 0 -> 2
- net /EN: track 8.79 -> 41.2 mm, vias 0 -> 2
- net /MISO: track 122.4 -> 147.3 mm, vias 6 -> 5
- net Net-(J2-Pad6): track 0.00 -> 20.2 mm, vias 0 -> 3
- net /MOSI: track 144.9 -> 163.2 mm, vias 6 -> 5
- net Net-(JP5-Pad2): track 5.22 -> 22.9 mm, vias 0 -> 2
- net /SD_CS: track 108.4 -> 94.1 mm
- net Net-(J5-Pad1): track 6.22 -> 16.8 mm
- net /SCLK: track 124.8 -> 132.3 mm, vias 8 -> 6
- net Net-(D15-Pad2): track 0.00 -> 6.15 mm
- net Net-(D11-Pad2): track 0.00 -> 5.70 mm
- net Net-(R23-Pad2): track 0.33 -> 5.53 mm
- net +3V3: track 90.0 -> 93.1 mm
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
Commit message: pcb update
Parts:
- moved J8 22.6 mm to (181.4, 87.7), turned to 90 degrees
- moved J6 20.7 mm to (181.4, 100.8), turned to 90 degrees
- moved D10 16.0 mm to (175.3, 103.1), turned to 0 degrees
- moved D15 15.7 mm to (175.7, 85.5), turned to 90 degrees
- moved R33 15.4 mm to (161.2, 85.2), turned to 90 degrees
- moved R30 15.4 mm to (161.5, 101.3), turned to 180 degrees
- moved D14 15.1 mm to (176.1, 89.0), turned to 0 degrees
- moved R35 13.8 mm to (161.5, 99.8), turned to 180 degrees
- moved R28 13.8 mm to (162.7, 85.2), turned to 90 degrees
- moved R27 13.8 mm to (172.0, 103.1), turned to 180 degrees
- moved J7 13.5 mm to (181.4, 94.3), turned to 90 degrees
- moved D11 13.2 mm to (175.9, 98.9), turned to 90 degrees
- moved D12 13.0 mm to (164.7, 101.3), turned to 0 degrees
- moved R29 12.4 mm to (164.1, 85.2), turned to 90 degrees
- moved Q5 12.1 mm to (172.9, 85.7), turned to 0 degrees
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Connections:
- Q3 pad 1: Net-(Q3-Pad1) -> /Buzzer
- U3 pad 10: /FLASH_CS -> /SD_CS
- U3 pad 11: /IMU_CS -> /Nuke2
- U3 pad 12: Net-(Q3-Pad1) -> /Nuke1
- U3 pad 13: /Nuke2 -> /MAG_CS
- U3 pad 14: /Nuke1 -> /IMU_CS
- U3 pad 23: /MAG_CS -> /FLASH_CS
- U3 pad 24: /LORA_CS -> /Buzzer
- U3 pad 27: /RADIO_TX -> /RADIO_RX
- U3 pad 28: /RADIO_RX -> /RADIO_TX
- U3 pad 29: /SD_CS -> /LORA_CS
Routing:
- net /FLASH_CS: track 3.34 -> 88.2 mm
- net /LORA_CS: track 2.80 -> 85.0 mm, vias 1 -> 0
- net /Buzzer: track 0.00 -> 82.0 mm
- net /Cont1: track 0.00 -> 65.2 mm, vias 0 -> 2
- net /Cont2: track 0.00 -> 63.6 mm, vias 0 -> 2
- net /Nuke2: track 0.00 -> 56.7 mm
- net /Nuke1: track 0.00 -> 55.1 mm
- net /IMU_CS: track 3.21 -> 52.7 mm
- net /MAG_CS: track 3.82 -> 52.0 mm
- net Net-(D10-Pad2): track 29.4 -> 0.00 mm, vias 1 -> 0
- net /SD_CS: track 94.1 -> 69.8 mm
- net Net-(D14-Pad2): track 15.7 -> 0.00 mm, vias 1 -> 0
- net GND: track 40.9 -> 30.1 mm
- net /RADIO_RX: track 48.2 -> 38.3 mm, vias 1 -> 0
- net /RADIO_TX: track 44.2 -> 37.8 mm
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
Commit message: pcb update
Parts:
- removed JP3, JP4: SolderJumper_3_Open, Jumper:SolderJumper-3_P2.0mm_Open_TrianglePad1.0x1.5mm_NumberLabels
- moved J7 19.6 mm to (166.0, 106.4), turned to 0 degrees
- moved D16 8.47 mm to (167.8, 91.9)
- moved R35 8.47 mm to (164.5, 91.9)
- moved D10 4.71 mm to (175.9, 98.5)
- moved Q4 4.71 mm to (172.8, 95.6)
- moved R27 4.71 mm to (172.6, 98.5)
- moved D11 3.69 mm to (175.7, 95.2)
- moved J6 3.33 mm to (181.4, 97.5)
- moved J8 3.25 mm to (181.4, 91.0)
- moved D12 3.07 mm to (167.5, 100.1)
- moved R30 3.07 mm to (164.3, 100.1)
- moved Q5 2.79 mm to (172.5, 88.5)
- moved R32 2.79 mm to (172.3, 91.7)
- moved D14 2.79 mm to (175.7, 91.8)
- moved D15 2.79 mm to (175.4, 88.2)
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Connections:
- D10 pad 2: Net-(D10-Pad2) -> /nukes/External_Supply
- D14 pad 2: Net-(D14-Pad2) -> /nukes/External_Supply
- J6 pad 1: Net-(D10-Pad2) -> /nukes/External_Supply
- J8 pad 1: Net-(D14-Pad2) -> /nukes/External_Supply
- U3 pad 11: /Nuke2 -> /Nuke1
- U3 pad 12: /Nuke1 -> /Nuke2
Routing:
- net /nukes/External_Supply: track 9.03 -> 49.1 mm
- net /Nuke1: track 55.1 -> 88.9 mm, vias 0 -> 2
- net /Cont1: track 65.2 -> 89.7 mm
- net /Nuke2: track 56.7 -> 79.3 mm, vias 0 -> 2
- net Net-(D15-Pad2): track 0.00 -> 21.6 mm
- net Net-(D11-Pad2): track 0.54 -> 20.6 mm
- net /Cont2: track 63.6 -> 77.9 mm
- net Net-(R29-Pad1): track 0.00 -> 13.0 mm
- net Net-(D11-Pad1): track 0.00 -> 5.93 mm
- net Net-(D15-Pad1): track 0.65 -> 6.46 mm
- net GND: track 30.1 -> 25.1 mm
- net Net-(R24-Pad2): track 0.00 -> 4.89 mm
- net Net-(R34-Pad1): track 0.00 -> 4.40 mm
- net Net-(J4-Pad1): track 15.9 -> 18.1 mm
- net Net-(D14-Pad1): track 0.07 -> 1.88 mm
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- added copper zone on B.Cu, net GND
- added copper zone on F.Cu, net GND

Commit message: pcb update
Routing:
- added copper zone on In2.Cu, net GND
- removed copper zone on In1.Cu, net GND
