File: power.sch (KiCad schematic (older format))
At the start: 6 parts

Commit message: Fixed power capacitors and added chip footprint
Parts:
- removed C?: 10u, Capacitor_SMD:CP_Elec_4x5.4, symbol Device:C
- removed C?: 10u, Capacitor_SMD:C_0201_0603Metric, symbol Device:C
- U?: footprint (none) -> Package_SON:Texas_S-PVSON-N10_ThermalVias; symbol iclr:TPS63031 -> Mainboard-rescue:TPS63031-iclr
Connections:
- wire segments 31 -> 27
Other:
- moved on the sheet: C?
Changed lines of the file:
@@
 EESchema Schematic File Version 4
 LIBS:Mainboard-cache
-EELAYER 30 0
+EELAYER 29 0
 EELAYER END
 $Descr A4 11693 8268
@@
 	1    0    0    -1
 $EndComp
-$Comp
-L Device:C C?
-U 1 1 5DBA4ED0
-P 6550 4300
-F 0 "C?" H 6665 4346 50  0000 L CNN
-F 1 "10u" H 6665 4255 50  0000 L CNN
-F 2 "Capacitor_SMD:CP_Elec_4x5.4" H 6588 4150 50  0001 C CNN
-F 3 "~" H 6550 4300 50  0001 C CNN
-	1    6550 4300
-	1    0    0    -1
-$EndComp
 Wire Wire Line
 	6400 3800 6550 3800
@@
 Wire Wire Line
 	6550 3800 6700 3800
-Wire Wire Line
-	6550 4450 6550 4700
-$Comp
-L iclr:TPS63031 U?
-U 1 1 5DBADF56
-P 5900 3400
-F 0 "U?" H 5900 3450 50  0000 C CNN
-F 1 "TPS63031" H 5900 3350 50  0000 C CNN
-F 2 "" H 5900 3400 50  0001 C CNN
-F 3 "" H 5900 3400 50  0001 C CNN
-	1    5900 3400
-	1    0    0    -1
-$EndComp
 Wire Wire Line
 	6350 3600 6400 3600
@@
 Connection ~ 5400 4000
 $Comp
-L Device:C C?
-U 1 1 5DBBD700
-P 5150 4050
-F 0 "C?" H 5265 4096 50  0000 L CNN
-F 1 "10u" H 5265 4005 50  0000 L CNN
-F 2 "Capacitor_SMD:C_0201_0603Metric" H 5188 3900 50  0001 C CNN
-F 3 "~" H 5150 4050 50  0001 C CNN
-	1    5150 4050
+L power:GND #PWR?
+U 1 1 5DBBE1E1
+P 5000 4250
+F 0 "#PWR?" H 5000 4000 50  0001 C CNN
+F 1 "GND" H 5005 4077 50  0000 C CNN
+F 2 "" H 5000 4250 50  0001 C CNN
+F 3 "" H 5000 4250 50  0001 C CNN
+	1    5000 4250
 	1    0    0    -1
 $EndComp
-Wire Wire Line
-	5400 3900 5150 3900
-Connection ~ 5400 3900
-$Comp
-L power:GND #PWR?
-U 1 1 5DBBE1E1
-P 5150 4300
-F 0 "#PWR?" H 5150 4050 50  0001 C CNN
-F 1 "GND" H 5155 4127 50  0000 C CNN
-F 2 "" H 5150 4300 50  0001 C CNN
-F 3 "" H 5150 4300 50  0001 C CNN
-	1    5150 4300
-	1    0    0    -1
-$EndComp
-Wire Wire Line
-	5150 4200 5150 4250
 $Comp
 L power:VDD #PWR?
 U 1 1 5DBCE035
-P 4650 3800
-F 0 "#PWR?" H 4650 3650 50  0001 C CNN
-F 1 "VDD" H 4667 3973 50  0000 C CNN
-F 2 "" H 4650 3800 50  0001 C CNN
-F 3 "" H 4650 3800 50  0001 C CNN
-	1    4650 3800
+P 5000 3750
+F 0 "#PWR?" H 5000 3600 50  0001 C CNN
+F 1 "VDD" H 5017 3923 50  0000 C CNN
+F 2 "" H 5000 3750 50  0001 C CNN
+F 3 "" H 5000 3750 50  0001 C CNN
+	1    5000 3750
 	1    0    0    -1
 $EndComp
@@
 L Device:C C?
 U 1 1 5DBCE6FA
-P 4800 4050
-F 0 "C?" H 4915 4096 50  0000 L CNN
-F 1 "10u" H 4915 4005 50  0000 L CNN
-F 2 "Capacitor_SMD:CP_Elec_4x5.4" H 4838 3900 50  0001 C CNN
-F 3 "~" H 4800 4050 50  0001 C CNN
-	1    4800 4050
+P 5000 4050
+F 0 "C?" H 5115 4096 50  0000 L CNN
+F 1 "10u" H 5115 4005 50  0000 L CNN
+F 2 "Capacitor_SMD:CP_Elec_4x5.4" H 5038 3900 50  0001 C CNN
+F 3 "~" H 5000 4050 50  0001 C CNN
+	1    5000 4050
 	1    0    0    -1
 $EndComp
 Wire Wire Line
-	4800 4200 4800 4250
+	5000 4200 5000 4250
 Wire Wire Line
-	4800 4250 5150 4250
-Connection ~ 5150 4250
+	5000 3750 5000 3800
 Wire Wire Line
-	5150 4250 5150 4300
+	5000 3900 5000 3800
+Connection ~ 5000 3800
 Wire Wire Line
-	4650 3800 4800 3800
+	5000 3800 5450 3800
+$Comp
+L Mainboard-rescue:TPS63031-iclr U?
+U 1 1 5DBADF56
+P 5900 3400
+AR Path="/5DBADF56" Ref="U?"  Part="1"
+AR Path="/5DB9F80E/5DBADF56" Ref="U?"  Part="1"
+F 0 "U?" H 5900 3450 50  0000 C CNN
+F 1 "TPS63031" H 5900 3350 50  0000 C CNN
+F 2 "Package_SON:Texas_S-PVSON-N10_ThermalVias" H 5900 3400 50  0001 C CNN
+F 3 "" H 5900 3400 50  0001 C CNN
+	1    5900 3400
+	1    0    0    -1
+$EndComp
 Wire Wire Line
-	4800 3900 4800 3800
-Connection ~ 4800 3800
-Wire Wire Line
-	4800 3800 5450 3800
+	6550 4150 6550 4700
 $EndSCHEMATC

Commit message: Add files via upload
Parts:
- removed U?: TPS63031, Package_SON:Texas_S-PVSON-N10_ThermalVias, symbol Mainboard-rescue:TPS63031-iclr
- added U8: TPS63031, symbol iclr:TPS63031
- gave numbers to parts that had none: 3
Changed lines of the file:
@@
 $EndDescr
 $Comp
-L pspice:INDUCTOR L?
+L pspice:INDUCTOR L2
 U 1 1 5DBA17F7
 P 5900 3200
-F 0 "L?" H 5900 3415 50  0000 C CNN
+F 0 "L2" H 5900 3415 50  0000 C CNN
 F 1 "1u5" H 5900 3324 50  0000 C CNN
 F 2 "Inductor_SMD:L_Taiyo-Yuden_NR-30xx" H 5900 3200 50  0001 C CNN
@@
 Connection ~ 6400 3800
 $Comp
-L power:+3V3 #PWR?
+L power:+3V3 #PWR052
 U 1 1 5DBA4350
 P 6700 3800
-F 0 "#PWR?" H 6700 3650 50  0001 C CNN
+F 0 "#PWR052" H 6700 3650 50  0001 C CNN
 F 1 "+3V3" H 6715 3973 50  0000 C CNN
 F 2 "" H 6700 3800 50  0001 C CNN
@@
 	6400 3800 6550 3800
 $Comp
-L Device:C C?
+L Device:C C11
 U 1 1 5DBA6514
 P 6550 4000
-F 0 "C?" H 6665 4046 50  0000 L CNN
+F 0 "C11" H 6665 4046 50  0000 L CNN
 F 1 "10u" H 6665 3955 50  0000 L CNN
 F 2 "Capacitor_SMD:CP_Elec_4x5.4" H 6588 3850 50  0001 C CNN
@@
 	5800 4700 6550 4700
 $Comp
-L power:GND #PWR?
+L power:GND #PWR051
 U 1 1 5DBB0345
 P 5750 4700
-F 0 "#PWR?" H 5750 4450 50  0001 C CNN
+F 0 "#PWR051" H 5750 4450 50  0001 C CNN
 F 1 "GND" H 5755 4527 50  0000 C CNN
 F 2 "" H 5750 4700 50  0001 C CNN
@@
 Connection ~ 5400 4000
 $Comp
-L power:GND #PWR?
+L power:GND #PWR050
 U 1 1 5DBBE1E1
 P 5000 4250
-F 0 "#PWR?" H 5000 4000 50  0001 C CNN
+F 0 "#PWR050" H 5000 4000 50  0001 C CNN
 F 1 "GND" H 5005 4077 50  0000 C CNN
 F 2 "" H 5000 4250 50  0001 C CNN
@@
 $EndComp
 $Comp
-L power:VDD #PWR?
+L power:VDD #PWR049
 U 1 1 5DBCE035
 P 5000 3750
-F 0 "#PWR?" H 5000 3600 50  0001 C CNN
+F 0 "#PWR049" H 5000 3600 50  0001 C CNN
 F 1 "VDD" H 5017 3923 50  0000 C CNN
 F 2 "" H 5000 3750 50  0001 C CNN
@@
 $EndComp
 $Comp
-L Device:C C?
+L Device:C C10
 U 1 1 5DBCE6FA
 P 5000 4050
-F 0 "C?" H 5115 4096 50  0000 L CNN
+F 0 "C10" H 5115 4096 50  0000 L CNN
 F 1 "10u" H 5115 4005 50  0000 L CNN
 F 2 "Capacitor_SMD:CP_Elec_4x5.4" H 5038 3900 50  0001 C CNN
@@
 Wire Wire Line
 	5000 3800 5450 3800
+Wire Wire Line
+	6550 4150 6550 4700
 $Comp
-L Mainboard-rescue:TPS63031-iclr U?
-U 1 1 5DBADF56
-P 5900 3400
-AR Path="/5DBADF56" Ref="U?"  Part="1"
-AR Path="/5DB9F80E/5DBADF56" Ref="U?"  Part="1"
-F 0 "U?" H 5900 3450 50  0000 C CNN
-F 1 "TPS63031" H 5900 3350 50  0000 C CNN
-F 2 "Package_SON:Texas_S-PVSON-N10_ThermalVias" H 5900 3400 50  0001 C CNN
-F 3 "" H 5900 3400 50  0001 C CNN
-	1    5900 3400
+L iclr:TPS63031 U8
+U 1 1 5DE04FA4
+P 5900 4000
+F 0 "U8" H 5733 4665 50  0000 C CNN
+F 1 "TPS63031" H 5733 4574 50  0000 C CNN
+F 2 "" H 5900 4600 50  0001 C CNN
+F 3 "" H 5900 4600 50  0001 C CNN
+	1    5900 4000
 	1    0    0    -1
 $EndComp
-Wire Wire Line
-	6550 4150 6550 4700
 $EndSCHEMATC

Commit message: Updated TPS63031 fp
Parts:
- U8: footprint (none) -> iclr:VSON-10-1EP_2.5x2.5mm_Pitch0.5mm_ThermalPad
Changed lines of the file:
@@
 EESchema Schematic File Version 4
 LIBS:Mainboard-cache
-EELAYER 30 0
+EELAYER 29 0
 EELAYER END
 $Descr A4 11693 8268
@@
 F 0 "U8" H 5733 4665 50  0000 C CNN
 F 1 "TPS63031" H 5733 4574 50  0000 C CNN
-F 2 "" H 5900 4600 50  0001 C CNN
+F 2 "iclr:VSON-10-1EP_2.5x2.5mm_Pitch0.5mm_ThermalPad" H 5900 4600 50  0001 C CNN
 F 3 "" H 5900 4600 50  0001 C CNN
 	1    5900 4000

Commit message: Add files via upload
Parts:
- added C12, C14, C16, C18, C20, C22, C24, C26, C28: 100nf, Capacitor_SMD:C_0603_1608Metric, symbol Device:C_Small
- added C13, C15, C17, C19, C21, C23, C25, C27, C29: 10uf, Capacitor_SMD:C_0603_1608Metric, symbol Device:C_Small
- added TP? (x2): TestPoint, symbol Connector:TestPoint
- U8: footprint iclr:VSON-10-1EP_2.5x2.5mm_Pitch0.5mm_ThermalPad -> iclr-hw:VSON-10-1EP_2.5x2.5mm_Pitch0.5mm_ThermalPad
Connections:
- net +3V3: now also C12.1, C13.1, C14.1, C15.1, C16.1, C17.1, C18.1, C19.1, C20.1, C21.1, C22.1, C23.1, C24.1, C25.1, C26.1, C27.1, C28.1, C29.1, TP?.1
- net GND: now also C12.2, C13.2, C14.2, C15.2, C16.2, C17.2, C18.2, C19.2, C20.2, C21.2, C22.2, C23.2, C24.2, C25.2, C26.2, C27.2, C28.2, C29.2
- net VDD: now also TP?.1

Commit message: Add files via upload
Parts:
- added J11: Conn_01x02_Male, Connector_JST:JST_PH_B2B-PH-K_1x02_P2.00mm_Vertical, symbol Connector:Conn_01x02_Male
- TP16, TP17: renamed from TP?; footprint (none) -> TestPoint:TestPoint_THTPad_1.0x1.0mm_Drill0.5mm
Connections:
- net GND: now also J11.2 (Pin_2)
- net VDD: now also J11.1 (Pin_1)
Changed lines of the file:
@@
-$EndComp
-$Comp
-L power:+3V3 #PWR?
-U 1 1 5E0765FC
-P 3950 5100
-AR Path="/5DE3360C/5E0765FC" Ref="#PWR?"  Part="1"
-AR Path="/5DB9F80E/5E0765FC" Ref="#PWR053"  Part="1"
-F 0 "#PWR053" H 3950 4950 50  0001 C CNN
-F 1 "+3V3" H 3965 5273 50  0000 C CNN
-F 2 "" H 3950 5100 50  0001 C CNN
-F 3 "" H 3950 5100 50  0001 C CNN
-	1    3950 5100
-	1    0    0    -1
 $EndComp
 $Comp
@@
 	3800 5250 3800 5150
 Wire Wire Line
-	3800 5150 3950 5150
-Wire Wire Line
 	4100 5150 4100 5250
-Wire Wire Line
-	3950 5100 3950 5150
-Connection ~ 3950 5150
-Wire Wire Line
-	3950 5150 4100 5150
 Wire Wire Line
 	3800 5450 3800 5550
@@
 	7650 5550 7650 5450
 $Comp
-L power:GND #PWR?
-U 1 1 5E084A03
-P 3950 5650
-AR Path="/5DE3360C/5E084A03" Ref="#PWR?"  Part="1"
-AR Path="/5DB9F80E/5E084A03" Ref="#PWR055"  Part="1"
-F 0 "#PWR055" H 3950 5400 50  0001 C CNN
-F 1 "GND" H 3955 5477 50  0000 C CNN
-F 2 "" H 3950 5650 50  0001 C CNN
-F 3 "" H 3950 5650 50  0001 C CNN
-	1    3950 5650
-	1    0    0    -1
-$EndComp
-$Comp
 L Device:C_Small C?
 U 1 1 5E084A09
@@
 	7950 5250 7950 5150
 Wire Wire Line
-	8250 5150 8250 5250
-Wire Wire Line
 	7950 5450 7950 5550
-Wire Wire Line
-	8250 5550 8250 5450
 Connection ~ 4100 5150
 Wire Wire Line
@@
 Wire Wire Line
 	7350 5550 7650 5550
-Wire Wire Line
-	3800 5550 3950 5550
-Wire Wire Line
-	3950 5650 3950 5550
-Connection ~ 3950 5550
-Wire Wire Line
-	3950 5550 4100 5550
-Wire Wire Line
-	7950 5550 8250 5550
 Wire Wire Line
 	7950 5150 8250 5150
@@
 	8250 5150 8550 5150
 Connection ~ 8550 5150
-Wire Wire Line
-	8250 5550 8550 5550
 Connection ~ 8550 5550
 Wire Wire Line
@@
 P 5000 3800
 AR Path="/5E403DEA" Ref="TP?"  Part="1"
-AR Path="/5DB9F80E/5E403DEA" Ref="TP?"  Part="1"
-F 0 "TP?" V 4954 3988 50  0000 L CNN
+AR Path="/5DB9F80E/5E403DEA" Ref="TP16"  Part="1"
+F 0 "TP16" V 4954 3988 50  0000 L CNN
 F 1 "TestPoint" V 5045 3988 50  0000 L CNN
-F 2 "" H 5200 3800 50  0001 C CNN
+F 2 "TestPoint:TestPoint_THTPad_1.0x1.0mm_Drill0.5mm" H 5200 3800 50  0001 C CNN
 F 3 "~" H 5200 3800 50  0001 C CNN
 	1    5000 3800
@@
 P 6700 3800
 AR Path="/5E4076DE" Ref="TP?"  Part="1"
-AR Path="/5DB9F80E/5E4076DE" Ref="TP?"  Part="1"
-F 0 "TP?" V 6654 3988 50  0000 L CNN
+AR Path="/5DB9F80E/5E4076DE" Ref="TP17"  Part="1"
+F 0 "TP17" V 6654 3988 50  0000 L CNN
 F 1 "TestPoint" V 6745 3988 50  0000 L CNN
-F 2 "" H 6900 3800 50  0001 C CNN
+F 2 "TestPoint:TestPoint_THTPad_1.0x1.0mm_Drill0.5mm" H 6900 3800 50  0001 C CNN
 F 3 "~" H 6900 3800 50  0001 C CNN
 	1    6700 3800
 	0    1    1    0
 $EndComp
+$Comp
+L Connector:Conn_01x02_Male J11
+U 1 1 5DE7E179
+P 3700 3350
+F 0 "J11" V 3762 3394 50  0000 L CNN
+F 1 "Conn_01x02_Male" V 3853 3394 50  0000 L CNN
+F 2 "Connector_JST:JST_PH_B2B-PH-K_1x02_P2.00mm_Vertical" H 3700 3350 50  0001 C CNN
+F 3 "~" H 3700 3350 50  0001 C CNN
+	1    3700 3350
+	0    1    1    0
+$EndComp
+$Comp
+L power:VDD #PWR062
+U 1 1 5DE7F5AD
+P 3700 3650
+F 0 "#PWR062" H 3700 3500 50  0001 C CNN
+F 1 "VDD" V 3717 3778 50  0000 L CNN
+F 2 "" H 3700 3650 50  0001 C CNN
+F 3 "" H 3700 3650 50  0001 C CNN
+	1    3700 3650
+	0    1    1    0
+$EndComp
+Wire Wire Line
+	3700 3550 3700 3650
+$Comp
+L power:GND #PWR059
+U 1 1 5DE8310C
+P 3600 3650
+F 0 "#PWR059" H 3600 3400 50  0001 C CNN
+F 1 "GND" H 3605 3477 50  0000 C CNN
+F 2 "" H 3600 3650 50  0001 C CNN
+F 3 "" H 3600 3650 50  0001 C CNN
+	1    3600 3650
+	1    0    0    -1
+$EndComp
+Wire Wire Line
+	3600 3650 3600 3550
+Wire Wire Line
+	8250 5250 8250 5150
+Wire Wire Line
+	7950 5550 8250 5550
+Connection ~ 8250 5150
+Wire Wire Line
+	8250 5450 8250 5550
+Connection ~ 8250 5550
+Wire Wire Line
+	8250 5550 8550 5550
+Wire Wire Line
+	3800 5550 4100 5550
+Wire Wire Line
+	3800 5150 4100 5150
+$Comp
+L Mainboard-cache:+3.3V #PWR0106
+U 1 1 5E4CE71E
+P 3800 5150
+F 0 "#PWR0106" H 3800 5000 50  0001 C CNN
+F 1 "+3.3V" H 3815 5323 50  0000 C CNN
+F 2 "" H 3800 5150 50  0001 C CNN
+F 3 "" H 3800 5150 50  0001 C CNN
+	1    3800 5150
+	1    0    0    -1
+$EndComp
+Connection ~ 3800 5150
+$Comp
+L power:GND #PWR0107
+U 1 1 5E4CEA96
+P 8850 5550
+F 0 "#PWR0107" H 8850 5300 50  0001 C CNN
+F 1 "GND" H 8855 5377 50  0000 C CNN
+F 2 "" H 8850 5550 50  0001 C CNN
+F 3 "" H 8850 5550 50  0001 C CNN
+	1    8850 5550
+	1    0    0    -1
+$EndComp
+Connection ~ 8850 5550
 $EndSCHEMATC

Commit message: routed almost all 3.3
Parts:
- added H1, H2, H3, H4: MountingHole_Pad, MountingHole:MountingHole_3.2mm_M3_DIN965_Pad, symbol Mechanical:MountingHole_Pad
- U8: symbol iclr:TPS63031 -> Mainboard-rescue:TPS63031-iclr
Connections:
- net GND: now also H1.1, H2.1, H3.1, H4.1
Changed lines of the file:
@@
 EESchema Schematic File Version 4
-LIBS:Mainboard-cache
 EELAYER 30 0
 EELAYER END
@@
 	6550 4150 6550 4700
 $Comp
-L iclr:TPS63031 U8
+L Mainboard-rescue:TPS63031-iclr U8
 U 1 1 5DE04FA4
 P 5900 4000
@@
 	3800 5150 4100 5150
 $Comp
-L Mainboard-cache:+3.3V #PWR0106
+L Mainboard-rescue:+3.3V-Mainboard-cache #PWR0106
 U 1 1 5E4CE71E
 P 3800 5150
+AR Path="/5E4CE71E" Ref="#PWR0106"  Part="1"
+AR Path="/5DB9F80E/5E4CE71E" Ref="#PWR0106"  Part="1"
 F 0 "#PWR0106" H 3800 5000 50  0001 C CNN
 F 1 "+3.3V" H 3815 5323 50  0000 C CNN
@@
 $EndComp
 Connection ~ 8850 5550
+$Comp
+L Mechanical:MountingHole_Pad H2
+U 1 1 5E1B83DE
+P 8300 3950
+F 0 "H2" H 8400 3999 50  0000 L CNN
+F 1 "MountingHole_Pad" H 8400 3908 50  0000 L CNN
+F 2 "MountingHole:MountingHole_3.2mm_M3_DIN965_Pad" H 8300 3950 50  0001 C CNN
+F 3 "~" H 8300 3950 50  0001 C CNN
+	1    8300 3950
+	1    0    0    -1
+$EndComp
+$Comp
+L Mechanical:MountingHole_Pad H1
+U 1 1 5E1B8AC2
+P 8050 3950
+F 0 "H1" H 8150 3999 50  0000 L CNN
+F 1 "MountingHole_Pad" H 8150 3908 50  0000 L CNN
+F 2 "MountingHole:MountingHole_3.2mm_M3_DIN965_Pad" H 8050 3950 50  0001 C CNN
+F 3 "~" H 8050 3950 50  0001 C CNN
+	1    8050 3950
+	1    0    0    -1
+$EndComp
+$Comp
+L Mechanical:MountingHole_Pad H3
+U 1 1 5E1BE159
+P 8550 3950
+F 0 "H3" H 8650 3999 50  0000 L CNN
+F 1 "MountingHole_Pad" H 8650 3908 50  0000 L CNN
+F 2 "MountingHole:MountingHole_3.2mm_M3_DIN965_Pad" H 8550 3950 50  0001 C CNN
+F 3 "~" H 8550 3950 50  0001 C CNN
+	1    8550 3950
+	1    0    0    -1
+$EndComp
+$Comp
+L Mechanical:MountingHole_Pad H4
+U 1 1 5E1C0B92
+P 8800 3950
+F 0 "H4" H 8900 3999 50  0000 L CNN
+F 1 "MountingHole_Pad" H 8900 3908 50  0000 L CNN
+F 2 "MountingHole:MountingHole_3.2mm_M3_DIN965_Pad" H 8800 3950 50  0001 C CNN
+F 3 "~" H 8800 3950 50  0001 C CNN
+	1    8800 3950
+	1    0    0    -1
+$EndComp
+Wire Wire Line
+	8050 4050 8300 4050
+Connection ~ 8300 4050
+Wire Wire Line
+	8300 4050 8550 4050
+Connection ~ 8550 4050
+Wire Wire Line
+	8550 4050 8800 4050
+Wire Wire Line
+	8050 4050 7900 4050
+Wire Wire Line
+	7900 4050 7900 4150
+Connection ~ 8050 4050
+$Comp
+L power:GND #PWR027
+U 1 1 5E1C87F6
+P 7900 4150
+F 0 "#PWR027" H 7900 3900 50  0001 C CNN
+F 1 "GND" H 7905 3977 50  0000 C CNN
+F 2 "" H 7900 4150 50  0001 C CNN
+F 3 "" H 7900 4150 50  0001 C CNN
+	1    7900 4150
+	1    0    0    -1
+$EndComp
 $EndSCHEMATC

Commit message: update
Changed lines of the file:
@@
 L power:VDD #PWR049
 U 1 1 5DBCE035
-P 5000 3750
-F 0 "#PWR049" H 5000 3600 50  0001 C CNN
-F 1 "VDD" H 5017 3923 50  0000 C CNN
-F 2 "" H 5000 3750 50  0001 C CNN
-F 3 "" H 5000 3750 50  0001 C CNN
-	1    5000 3750
+P 5150 3750
+F 0 "#PWR049" H 5150 3600 50  0001 C CNN
+F 1 "VDD" H 5167 3923 50  0000 C CNN
+F 2 "" H 5150 3750 50  0001 C CNN
+F 3 "" H 5150 3750 50  0001 C CNN
+	1    5150 3750
 	1    0    0    -1
 $EndComp
@@
 	5000 4200 5000 4250
 Wire Wire Line
-	5000 3750 5000 3800
-Wire Wire Line
 	5000 3900 5000 3800
 Connection ~ 5000 3800
 Wire Wire Line
-	5000 3800 5450 3800
+	5000 3800 5150 3800
 Wire Wire Line
 	6550 4150 6550 4700
@@
 	1    0    0    -1
 $EndComp
+Wire Wire Line
+	5150 3750 5150 3800
+Connection ~ 5150 3800
+Wire Wire Line
+	5150 3800 5450 3800
 $EndSCHEMATC
