File: revert.kicad_pcb (KiCad board)
At the start: 4 copper layers, 100 x 60 mm, 317 parts, among them J1 USB_B_Micro, J10 Conn_01x02_Male, J11 Conn_01x02_Male, J12 Conn_01x02_Male, J2 8P8C_LED, J3 Micro_SD_Card_Det, J4 Conn_Coaxial, J5 Conn_Coaxial, J6 Screw_Terminal_01x02, J7 Screw_Terminal_01x02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

Commit message: update
Parts:
- removed D17: USB_LED, LED_SMD:LED_0603_1608Metric_Castellated
- added USB: USB_LED, LED_SMD:LED_0603_1608Metric_Castellated, F.Cu at (116.3, 106.1)
- renumbered TP10 to 10, TP11 to 11, TP12 to 12, TP13 to 13, TP14 to 14, TP15 to 15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
