File: gps.sch (KiCad schematic (older format))
At the start: 6 parts, among them J4 Conn_Coaxial, U6 MAX-M8Q

Commit message: update
Parts:
- R24: value 10k -> 10K
Changed lines of the file:
@@
 P 5000 4450
 F 0 "R24" V 5207 4450 50  0000 C CNN
-F 1 "10k" V 5116 4450 50  0000 C CNN
+F 1 "10K" V 5116 4450 50  0000 C CNN
 F 2 "Resistor_SMD:R_0603_1608Metric" V 4930 4450 50  0001 C CNN
 F 3 "~" H 5000 4450 50  0001 C CNN
