File: radio.sch (KiCad schematic (older format))
At the start: 3 parts

Commit message: Add files via upload
Parts:
- removed C?: 100n, Capacitors_SMD:C_0603, symbol Device:C
- gave numbers to parts that had none: 2
Changed lines of the file:
@@
 $EndDescr
 $Comp
-L RF_Module:RFM95W-868S2 U?
+L RF_Module:RFM95W-868S2 U11
 U 1 1 5DE3478D
 P 5650 3750
-F 0 "U?" H 6050 4350 50  0000 C CNN
+F 0 "U11" H 6050 4350 50  0000 C CNN
 F 1 "RFM95W-868S2" H 6050 4250 50  0000 C CNN
 F 2 "RF_Module:HOPERF_RFM9XW_SMD" H 2350 5400 50  0001 C CNN
@@
 $EndComp
 $Comp
-L Connector:Conn_Coaxial J?
+L Connector:Conn_Coaxial J5
 U 1 1 5DE351BF
 P 6750 3450
-F 0 "J?" H 6850 3425 50  0000 L CNN
+F 0 "J5" H 6850 3425 50  0000 L CNN
 F 1 "Conn_Coaxial" H 6850 3334 50  0000 L CNN
 F 2 "Connector_Coaxial:SMA_Molex_73251-1153_EdgeMount_Horizontal" H 6750 3450 50  0001 C CNN
@@
 	6150 3450 6550 3450
 $Comp
-L power:GND #PWR?
+L power:GND #PWR0102
 U 1 1 5DE36243
 P 6750 3700
-F 0 "#PWR?" H 6750 3450 50  0001 C CNN
+F 0 "#PWR0102" H 6750 3450 50  0001 C CNN
 F 1 "GND" H 6755 3527 50  0000 C CNN
 F 2 "" H 6750 3700 50  0001 C CNN
@@
 	6750 3700 6750 3650
 $Comp
-L power:GND #PWR?
+L power:GND #PWR0103
 U 1 1 5DE37EF9
 P 5750 4450
-F 0 "#PWR?" H 5750 4200 50  0001 C CNN
+F 0 "#PWR0103" H 5750 4200 50  0001 C CNN
 F 1 "GND" H 5755 4277 50  0000 C CNN
 F 2 "" H 5750 4450 50  0001 C CNN
@@
 	5650 4400 5750 4400
 $Comp
-L power:+3V3 #PWR?
+L power:+3V3 #PWR0104
 U 1 1 5DE3966F
 P 5650 3200
-F 0 "#PWR?" H 5650 3050 50  0001 C CNN
+F 0 "#PWR0104" H 5650 3050 50  0001 C CNN
 F 1 "+3V3" H 5665 3373 50  0000 C CNN
 F 2 "" H 5650 3200 50  0001 C CNN
@@
 Text HLabel 6150 4150 2    50   Output ~ 0
 ~INT
-$Comp
-L Device:C C?
-U 1 1 5DE3C0BF
-P 4200 3650
-F 0 "C?" H 4315 3696 50  0000 L CNN
-F 1 "100n" H 4315 3605 50  0000 L CNN
-F 2 "Capacitors_SMD:C_0603" H 4238 3500 50  0001 C CNN
-F 3 "~" H 4200 3650 50  0001 C CNN
-	1    4200 3650
-	1    0    0    -1
-$EndComp
-$Comp
-L power:+3V3 #PWR?
-U 1 1 5DE3CB60
-P 4200 3450
-F 0 "#PWR?" H 4200 3300 50  0001 C CNN
-F 1 "+3V3" H 4215 3623 50  0000 C CNN
-F 2 "" H 4200 3450 50  0001 C CNN
-F 3 "" H 4200 3450 50  0001 C CNN
-	1    4200 3450
-	1    0    0    -1
-$EndComp
-Wire Wire Line
-	4200 3450 4200 3500
-$Comp
-L power:GND #PWR?
-U 1 1 5DE3D454
-P 4200 3850
-F 0 "#PWR?" H 4200 3600 50  0001 C CNN
-F 1 "GND" H 4205 3677 50  0000 C CNN
-F 2 "" H 4200 3850 50  0001 C CNN
-F 3 "" H 4200 3850 50  0001 C CNN
-	1    4200 3850
-	1    0    0    -1
-$EndComp
-Wire Wire Line
-	4200 3850 4200 3800
 $EndSCHEMATC
