File: gsm_xbee/gsm_xbee.sch (KiCad schematic (older format))
At the start: 10 parts

Commit message: udpate
Parts:
- removed C?: 0.1uF, symbol Device:C_Small
- removed U?: TPD3E001DRLR, Package_TO_SOT_SMD:SOT-543, symbol Power_Protection:TPD3E001DRLR
- added C?: 22pF, symbol Device:C_Small
- added C?: 1uF, symbol Device:C_Small
- added C?: 100nF, symbol Device:C_Small
- added C?: 4.7uF, symbol Device:C_Small
- added D?: SP0503BAHT, Package_TO_SOT_SMD:SOT-143, symbol Power_Protection:SP0503BAHT
- added J?: Conn_01x02_Male, symbol Connector:Conn_01x02_Male
- added JP?: XBEE, XBEE, symbol iclr-hw:XBEE
Connections:
- net GND: now also C?.1, C?.1, C?.2, C?.2, D?.1 (A), J?.2 (Pin_2), JP?.10 (GND)
- net RXD: now also JP?.3 (DIN)
- net TXD: now also JP?.2 (DOUT)
- net USB_D+: now also D?.3 (K)
- net USB_D-: now also D?.4 (K)
- net USB_VBUS: now also C?.2, D?.2 (K)
- net VCC: now also U?.1 (VBAT), U?.42 (VBAT@1)
- net at R?.2, U?.14 (SIM_DATA): now also C?.1
- net at D?.5 (IO4), J?.C1 (VCC), U?.16 (VSIM): now also C?.2
- net at U?.49 (RESET): now also J?.1 (Pin_1)
- net at U?.56 (VRTC): now also C?.1
- net STATUS: now reaches U?.64 (NETLIGHT)
- new net +3V3: JP?.1 (VDD)
- no-connect marks 5 -> 4
Other:
- moved on the sheet: R?
