File: gsm_xbee/_autosave-gsm_xbee.sch (KiCad schematic (older format))
At the start: 30 parts

Commit message: update board
Connections:
- net RING: now also D?.1 (K)
- net RXD: now also D?.1 (K)
- net TXD: now also D?.1 (K)
Changed lines of the file:
@@
 	1    0    0    -1
 $EndComp
+Wire Wire Line
+	7600 4200 7850 4200
+Wire Wire Line
+	7600 4400 7850 4400
+Wire Wire Line
+	7600 4650 7850 4650
+Text Label 7850 4200 2    50   ~ 0
+RING
+Text Label 7850 4400 2    50   ~ 0
+RXD
+Text Label 7850 4650 2    50   ~ 0
+TXD
 $EndSCHEMATC
