File: BigRedButton/BigRedButton.kicad_sch (KiCad schematic)
At the start: 13 parts

Commit message: Added sd card and more changes
Parts:
- removed C? (x2): 100n, symbol Device:C_Small
- removed C?: 22u, symbol Device:C_Small
- removed R?: 10k, symbol Device:R_Small
- added C?: 4U7, symbol Device:C_Small
- added C?: 100nF, Capacitor_SMD:C_0603_1608Metric, symbol Device:C_Small
- added C?: 100n, symbol Device:C_Small
- added J?: Micro_SD_Card_Det, Connector_Card:microSD_HC_Hirose_DM3AT-SF-PEJM5, symbol Connector:Micro_SD_Card_Det_Hirose_DM3AT
- added P?: USB_C, Connector_USB:USB_C_Receptacle_GCT_USB4085, symbol Connector:USB_C_Receptacle
- added R? (x4): 5k1, symbol Device:R_Small
- added R?: 47k5, symbol Device:R_Small
- added R? (x3): 10K, Resistor_SMD:R_0603_1608Metric, symbol Device:R_Small
- added R?: 22k1, symbol Device:R_Small
- added R?: 2k, symbol Device:R_Small
- added R?: 10k, symbol Device:R_Small
- added U?: CP2102N-A01-GQFN28, Package_DFN_QFN:QFN-28-1EP_5x5mm_P0.5mm_EP3.35x3.35mm, symbol Interface_USB:CP2102N-A01-GQFN28
Connections:
- net +3V3: now also C?.2, C?.2, J?.4 (VDD), R?.1, R?.1, R?.1, R?.2, U?.6 (VDD), U?.7 (REGIN)
- net DTR: now also U?.28 (~DTR)
- net EN: now also C?.1, R?.2
- net GND: now also C?.1, C?.1, C?.2, J?.11 (SHIELD), J?.6 (VSS), P?.A1 (GND), P?.A12 (GND), P?.B1 (GND), P?.B12 (GND), P?.S1 (SHIELD), R?.1, R?.2, R?.2, R?.2, U?.29 (GND), U?.3 (GND)
- net IO0: now also R?.2
- net RTS: now also U?.24 (~RTS)
- net RX0: now also U?.25 (RXD)
- net TX0: now also U?.26 (TXD)
- new net: P?.A5 (CC1), R?.1
- new net: P?.B5 (CC2), R?.1
- new net: P?.A7 (D-), P?.B7 (D-), R?.2
- new net: R?.1, R?.2, U?.8 (VBUS)
- new net: P?.A6 (D+), P?.B6 (D+), R?.2
- new net: P?.A4 (VBUS), P?.A9 (VBUS), P?.B4 (VBUS), P?.B9 (VBUS)
- new net: R?.2, U?.9 (~RSTb)
- new net: R?.2, U?.11 (~SUSPENDb)
- new net D+: R?.1, U?.4 (D+)
- new net D-: R?.1, U?.5 (D-)
- new net MISO: J?.7 (DAT0)
- new net MOSI: J?.3 (CMD)
- new net SCLK: J?.5 (CLK)
- new net SD_CS: J?.2 (DAT3/CD), R?.1
- new net VBUS: R?.1
- no-connect marks 6 -> 35
Other:
- sheet Power ports: added none; removed DTR, RTS, RX0, TX0
- note added: "USBC STUFF"
- moved on the sheet: C?, Q?A, Q?B, R?, SW?, U?
