File: BigRedButton/power.kicad_sch (KiCad schematic)
At the start: 12 parts

Commit message: Added sd card and more changes
Parts:
- removed C?: 100n, symbol Device:C_Small
- removed C?: 4U7, symbol Device:C_Small
- removed P?: USB_C, Connector_USB:USB_C_Receptacle_GCT_USB4085, symbol Connector:USB_C_Receptacle
- removed R? (x4): 5k1, symbol Device:R_Small
- removed R?: 10k, symbol Device:R_Small
- removed R?: 2k, symbol Device:R_Small
- removed R?: 22k1, symbol Device:R_Small
- removed R?: 47k5, symbol Device:R_Small
- removed U?: CP2102N-A01-GQFN28, Package_DFN_QFN:QFN-28-1EP_5x5mm_P0.5mm_EP3.35x3.35mm, symbol Interface_USB:CP2102N-A01-GQFN28
Connections:
- no-connect marks 25 -> 0
Other:
- note removed: "USB STUFF"
