File: Bluetooth_Igniter_SANIC/power.sch (KiCad schematic (older format))
At the start: 13 parts, among them J4 Screw_Terminal_01x02, U5 TPS63060

Commit message: Small change
Parts:
- J4: footprint (none) -> iclrhw:PHOENIX_1757242
Changed lines of the file:
@@
 F 0 "J4" H 2568 1525 50  0000 C CNN
 F 1 "Screw_Terminal_01x02" H 2568 1616 50  0000 C CNN
-F 2 "" H 2650 1850 50  0001 C CNN
+F 2 "iclrhw:PHOENIX_1757242" H 2650 1850 50  0001 C CNN
 F 3 "~" H 2650 1850 50  0001 C CNN
 	1    2650 1850
@@
 Wire Wire Line
 	5150 3900 5200 3900
-Text Label 6950 3850 0    50   ~ 0
-PG
 Wire Wire Line
 	7150 3050 7500 3050
@@
 	1    0    0    -1
 $EndComp
+Text HLabel 7050 3850 2    50   Input ~ 0
+PG
+$Comp
+L power:VDD #PWR0102
+U 1 1 605331BA
+P 7000 1100
+F 0 "#PWR0102" H 7000 950 50  0001 C CNN
+F 1 "VDD" H 7015 1273 50  0000 C CNN
+F 2 "" H 7000 1100 50  0001 C CNN
+F 3 "" H 7000 1100 50  0001 C CNN
+	1    7000 1100
+	1    0    0    -1
+$EndComp
+$Comp
+L power:PWR_FLAG #FLG0101
+U 1 1 60534408
+P 7000 1100
+F 0 "#FLG0101" H 7000 1175 50  0001 C CNN
+F 1 "PWR_FLAG" H 7000 1273 50  0000 C CNN
+F 2 "" H 7000 1100 50  0001 C CNN
+F 3 "~" H 7000 1100 50  0001 C CNN
+	1    7000 1100
+	-1   0    0    1
+$EndComp
+$Comp
+L power:GND #PWR0103
+U 1 1 60538466
+P 8050 1100
+F 0 "#PWR0103" H 8050 850 50  0001 C CNN
+F 1 "GND" H 8055 927 50  0000 C CNN
+F 2 "" H 8050 1100 50  0001 C CNN
+F 3 "" H 8050 1100 50  0001 C CNN
+	1    8050 1100
+	1    0    0    -1
+$EndComp
+$Comp
+L power:PWR_FLAG #FLG0103
+U 1 1 60537967
+P 8050 1100
+F 0 "#FLG0103" H 8050 1175 50  0001 C CNN
+F 1 "PWR_FLAG" H 8050 1273 50  0000 C CNN
+F 2 "" H 8050 1100 50  0001 C CNN
+F 3 "~" H 8050 1100 50  0001 C CNN
+	1    8050 1100
+	1    0    0    -1
+$EndComp
