File: Bluetooth_Igniter_SANIC/usb.sch (KiCad schematic (older format))
At the start: 5 parts, among them J5 USB_C_Receptacle_USB2.0

Commit message: Small change
Parts:
- J5: footprint (none) -> Connector_USB:USB_C_Receptacle_XKB_U262-16XN-4BVC11
Changed lines of the file:
@@
 F 0 "J5" H 5207 4267 50  0000 C CNN
 F 1 "USB_C_Receptacle_USB2.0" H 5207 4176 50  0000 C CNN
-F 2 "" H 5250 3400 50  0001 C CNN
+F 2 "Connector_USB:USB_C_Receptacle_XKB_U262-16XN-4BVC11" H 5250 3400 50  0001 C CNN
 F 3 "https://www.usb.org/sites/default/files/documents/usb_type-c.zip" H 5250 3400 50  0001 C CNN
 	1    5100 3400
