File: Bluetooth_Igniter_SANIC/Bluetooth_ignite_receiver.kicad_pcb (KiCad board)
At the start: 2 copper layers, 73 x 30 mm, 71 parts, among them J1 Screw_Terminal_01x02, J10 Conn_01x02_Male, J2 Screw_Terminal_01x02, J3 Screw_Terminal_01x02, J4 Screw_Terminal_01x02, J5 USB_C_Receptacle_USB2.0, J6 Conn_01x02_Male, J7 Conn_01x02_Male, J8 Conn_01x04_Male, J9 Conn_01x07_Male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

Commit message: Forgot to connect a ground node on regulator. Fixed now
Routing:
- net GND: track 109.2 -> 113.9 mm
