File: Bluetooth_Igniter_SANIC/Bluetooth_ignite_receiver.sch (KiCad schematic (older format))
At the start: 24 parts, among them Q1 MMDT2222A, Q2 MMDT2222A, SW1 SW_Push, SW2 SW_Push, U1 CP2102N-A01-GQFN24, U2 ESP32-WROOM-32

Commit message: Small change
Parts:
- added D?: RX_LED, LED_SMD:LED_0603_1608Metric_Castellated, symbol Device:LED
- added D?: TX_LED, LED_SMD:LED_0603_1608Metric_Castellated, symbol Device:LED
- added R? (x2): 470, Resistor_SMD:R_0603_1608Metric, symbol Device:R_Small
- SW1, SW2: footprint (none) -> Button_Switch_SMD:SW_Push_1P1T_NO_CK_KMR2
Connections:
- net labels added: PG
- wire segments 91 -> 98
- no-connect marks 35 -> 34
Other:
- moved on the sheet: D1, D2, R3, R4, R5, U1

Commit message: Separate voltage supply for ESP32 and pyros
Parts:
- gave numbers to parts that had none: 4
Changed lines of the file:
@@
 Text Label 6750 4300 0    50   ~ 0
 Nuke1
-$Sheet
-S 9350 5350 1000 600
-U 603A281D
-F0 "pyros" 50
-F1 "pyros.sch" 50
-F2 "Cont1" I L 9350 5650 50
-F3 "Nuke2" I L 9350 5550 50
-F4 "Cont2" I L 9350 5750 50
-F5 "Nuke1" I L 9350 5450 50
-$EndSheet
 Connection ~ 5300 1300
 Wire Wire Line
@@
 	1400 3650 1400 4200
 $Comp
-L Device:R_Small R?
+L Device:R_Small R25
 U 1 1 605990BB
 P 7200 2500
-F 0 "R?" H 7259 2546 50  0000 L CNN
+F 0 "R25" H 7259 2546 50  0000 L CNN
 F 1 "470" H 7259 2455 50  0000 L CNN
 F 2 "Resistor_SMD:R_0603_1608Metric" H 7200 2500 50  0001 C CNN
@@
 $EndComp
 $Comp
-L Device:LED D?
+L Device:LED D13
 U 1 1 605990C1
 P 7200 2750
-F 0 "D?" V 7239 2632 50  0000 R CNN
+F 0 "D13" V 7239 2632 50  0000 R CNN
 F 1 "RX_LED" V 7148 2632 50  0000 R CNN
 F 2 "LED_SMD:LED_0603_1608Metric_Castellated" H 7200 2750 50  0001 C CNN
@@
 	7200 2900 7200 3050
 $Comp
-L Device:R_Small R?
+L Device:R_Small R24
 U 1 1 605B646E
 P 6650 2700
-F 0 "R?" H 6709 2746 50  0000 L CNN
+F 0 "R24" H 6709 2746 50  0000 L CNN
 F 1 "470" H 6709 2655 50  0000 L CNN
 F 2 "Resistor_SMD:R_0603_1608Metric" H 6650 2700 50  0001 C CNN
@@
 $EndComp
 $Comp
-L Device:LED D?
+L Device:LED D12
 U 1 1 605B6474
 P 6650 2950
-F 0 "D?" V 6689 2832 50  0000 R CNN
+F 0 "D12" V 6689 2832 50  0000 R CNN
 F 1 "TX_LED" V 6598 2832 50  0000 R CNN
 F 2 "LED_SMD:LED_0603_1608Metric_Castellated" H 6650 2950 50  0001 C CNN
@@
 Wire Wire Line
 	6400 2400 7200 2400
+$Sheet
+S 9350 5350 1000 600
+U 603A281D
+F0 "pyros" 50
+F1 "pyros.sch" 50
+F2 "Cont1" I L 9350 5650 50
+F3 "Nuke2" I L 9350 5550 50
+F4 "Cont2" I L 9350 5750 50
+F5 "Nuke1" I L 9350 5450 50
+$EndSheet
 $EndSCHEMATC

Commit message: small schematic changes
Parts:
- removed SW1, SW2: SW_Push, Button_Switch_SMD:SW_Push_1P1T_NO_CK_KMR2, symbol Switch:SW_Push
- added J6, J7: Conn_01x02_Male, Connector_PinHeader_2.54mm:PinHeader_1x02_P2.54mm_Vertical, symbol Connector:Conn_01x02_Male
Other:
- moved on the sheet: Q1A, Q2A, R1, R2

Commit message: need to fit pin headers in
Parts:
- added J8: Conn_01x04_Male, Connector_PinHeader_2.54mm:PinHeader_1x04_P2.54mm_Vertical, symbol Connector:Conn_01x04_Male
- added J9: Conn_01x07_Male, Connector_PinHeader_2.54mm:PinHeader_1x07_P2.54mm_Vertical, symbol Connector:Conn_01x07_Male
Connections:
- net labels added: CLK, CS, MISO, MOSI, SCL, SDA
- wire segments 98 -> 108
- no-connect marks 34 -> 28
Changed lines of the file:
@@
 NoConn ~ 6400 2500
 NoConn ~ 6400 2700
-NoConn ~ 6400 2800
 NoConn ~ 6400 2900
 NoConn ~ 6400 3000
@@
 NoConn ~ 6400 3300
 NoConn ~ 6400 3400
-NoConn ~ 6400 3500
-NoConn ~ 6400 3600
-NoConn ~ 6400 3700
-NoConn ~ 6400 3800
-NoConn ~ 6400 3900
 NoConn ~ 6400 4000
 NoConn ~ 6400 4200
@@
 Wire Wire Line
 	3400 4000 3700 4000
-Text Label 3700 3900 0    50   ~ 0
-RXD
-Text Label 3700 4000 0    50   ~ 0
-TXD
 Wire Wire Line
 	3400 3800 3700 3800
@@
 Wire Wire Line
 	1200 4700 1900 4700
-Text Label 3700 3800 0    50   ~ 0
+Text Label 3550 3800 0    50   ~ 0
 RTS
-Text Label 3700 4200 0    50   ~ 0
-DTR
 $Comp
 L Transistor_BJT:MMDT2222A Q1
@@
 Connection ~ 5300 1300
 Wire Wire Line
-	6400 4100 6750 4100
-Wire Wire Line
 	1500 750  1850 750
 Text Label 1850 750  0    50   ~ 0
-PG
-Text Label 6750 4100 0    50   ~ 0
 PG
 $Comp
@@
 Wire Wire Line
 	9850 1850 10150 1850
+Text Label 3550 3900 0    50   ~ 0
+RXD
+Text Label 3550 4000 0    50   ~ 0
+TXD
+Text Label 3550 4200 0    50   ~ 0
+DTR
+Wire Wire Line
+	6400 3700 6850 3700
+Wire Wire Line
+	6400 3800 6850 3800
+Text Label 6850 3700 2    50   ~ 0
+SDA
+Text Label 6850 3800 2    50   ~ 0
+SCL
+$Comp
+L Connector:Conn_01x04_Male J8
+U 1 1 60DB5E86
+P 3900 4000
+F 0 "J8" H 3872 3882 50  0000 R CNN
+F 1 "Conn_01x04_Male" H 3872 3973 50  0000 R CNN
+F 2 "Connector_PinHeader_2.54mm:PinHeader_1x04_P2.54mm_Vertical" H 3900 4000 50  0001 C CNN
+F 3 "~" H 3900 4000 50  0001 C CNN
+	1    3900 4000
+	-1   0    0    1
+$EndComp
+Wire Wire Line
+	3700 4200 3700 4100
+Wire Wire Line
+	6400 2800 6500 2800
+Wire Wire Line
+	6500 2800 6500 3400
+Wire Wire Line
+	6500 3400 6850 3400
+Wire Wire Line
+	6400 3500 6850 3500
+Wire Wire Line
+	6400 3600 6850 3600
+Wire Wire Line
+	6400 3900 6850 3900
+Text Label 6850 3400 2    50   ~ 0
+CS
+Text Label 6850 3500 2    50   ~ 0
+CLK
+Text Label 6850 3600 2    50   ~ 0
+MISO
+Text Label 6850 3900 2    50   ~ 0
+MOSI
+Wire Wire Line
+	6400 4100 6850 4100
+Text Label 6850 4100 2    50   ~ 0
+PG
+$Comp
+L Connector:Conn_01x07_Male J9
+U 1 1 60DCCD8A
+P 7050 3700
+F 0 "J9" H 7022 3632 50  0000 R CNN
+F 1 "Conn_01x07_Male" H 7022 3723 50  0000 R CNN
+F 2 "Connector_PinHeader_2.54mm:PinHeader_1x07_P2.54mm_Vertical" H 7050 3700 50  0001 C CNN
+F 3 "~" H 7050 3700 50  0001 C CNN
+	1    7050 3700
+	-1   0    0    1
+$EndComp
+Wire Wire Line
+	6850 4100 6850 4000
 $EndSCHEMATC

Commit message: update
Parts:
- C4, C5: value 1nF -> 0.1nF
Changed lines of the file:
@@
 P 9650 2200
 F 0 "C5" V 9421 2200 50  0000 C CNN
-F 1 "1nF" V 9512 2200 50  0000 C CNN
+F 1 "0.1nF" V 9512 2200 50  0000 C CNN
 F 2 "Capacitor_SMD:C_0603_1608Metric" H 9650 2200 50  0001 C CNN
 F 3 "~" H 9650 2200 50  0001 C CNN
@@
 P 9650 1200
 F 0 "C4" V 9421 1200 50  0000 C CNN
-F 1 "1nF" V 9512 1200 50  0000 C CNN
+F 1 "0.1nF" V 9512 1200 50  0000 C CNN
 F 2 "Capacitor_SMD:C_0603_1608Metric" H 9650 1200 50  0001 C CNN
 F 3 "~" H 9650 1200 50  0001 C CNN
