File: Pickle_Rick/Mainboard.sch (KiCad schematic (older format))
At the start: 81 parts, among them J10 Conn_01x02_Male, J12 Conn_01x02_Male, J2 8P8C_LED, J3 Micro_SD_Card_Det, J9 Conn_01x02_Male, Q1 MMDT2222A, Q3 PMV20ENR, U1 CP2102N-A01-GQFN24, U10 PCA9536D, U2 SN65HVD230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

Commit message: todo: change everything ᕙ(⇀‸↼‶)ᕗ
Parts:
- removed BZ1: Buzzer, Buzzer_Beeper:Buzzer_TDK_PS1240P02BT_D12.2mm_H6.5mm, symbol Device:Buzzer
- added J13: Conn_01x02, Connector_JST:JST_XH_B2B-XH-A_1x02_P2.50mm_Vertical, symbol Connector_Generic:Conn_01x02
Connections:
- net +3V3: now also J13.1 (Pin_1)
- net at D8.2 (A), R43.2: now also J13.2 (Pin_2)
Changed lines of the file:
@@
 F1 "power.sch" 50
 $EndSheet
-$Comp
-L Device:Buzzer BZ1
-U 1 1 5DBF25B1
-P 9000 2800
-F 0 "BZ1" H 9152 2829 50  0000 L CNN
-F 1 "Buzzer" H 9150 2750 50  0000 L CNN
-F 2 "Buzzer_Beeper:Buzzer_TDK_PS1240P02BT_D12.2mm_H6.5mm" V 8975 2900 50  0001 C CNN
-F 3 "~" V 8975 2900 50  0001 C CNN
-	1    9000 2800
-	1    0    0    -1
-$EndComp
 Wire Wire Line
 	5200 2750 5200 2650
@@
 Wire Wire Line
 	8900 2650 8750 2650
-Wire Wire Line
-	8900 2650 8900 2700
-Wire Wire Line
-	8900 2900 8900 2950
 Connection ~ 9600 4350
 $Comp
@@
 Wire Wire Line
 	7950 3550 8450 3550
+$Comp
+L Connector_Generic:Conn_01x02 J13
+U 1 1 60A3FF9E
+P 9100 2750
+F 0 "J13" H 9180 2742 50  0000 L CNN
+F 1 "Conn_01x02" H 9180 2651 50  0000 L CNN
+F 2 "Connector_JST:JST_XH_B2B-XH-A_1x02_P2.50mm_Vertical" H 9100 2750 50  0001 C CNN
+F 3 "~" H 9100 2750 50  0001 C CNN
+	1    9100 2750
+	1    0    0    -1
+$EndComp
+Wire Wire Line
+	8900 2650 8900 2750
+Wire Wire Line
+	8900 2850 8900 2950
 $EndSCHEMATC
