File: Pickle_Rick/radio.sch (KiCad schematic (older format))
At the start: 2 parts, among them J5 Conn_Coaxial, U11 RFM95W-868S2

Commit message: todo: change everything ᕙ(⇀‸↼‶)ᕗ
Parts:
- J5: footprint Connector_Coaxial:SMA_Molex_73251-1153_EdgeMount_Horizontal -> Connector_Coaxial:U.FL_Hirose_U.FL-R-SMT-1_Vertical
Changed lines of the file:
@@
 F 0 "J5" H 6850 3425 50  0000 L CNN
 F 1 "Conn_Coaxial" H 6850 3334 50  0000 L CNN
-F 2 "Connector_Coaxial:SMA_Molex_73251-1153_EdgeMount_Horizontal" H 6750 3450 50  0001 C CNN
+F 2 "Connector_Coaxial:U.FL_Hirose_U.FL-R-SMT-1_Vertical" H 6750 3450 50  0001 C CNN
 F 3 " ~" H 6750 3450 50  0001 C CNN
 	1    6750 3450
