File: Pickle_Rick/Mainboard.kicad_pcb (KiCad board)
At the start: 4 copper layers, 152 parts, among them J1 USB_C_Receptacle, J10 Conn_01x02_Male, J11 Conn_01x02_Male, J12 Conn_01x02_Male, J13 Conn_01x02, J14 Conn_01x02_Male, J2 8P8C_LED, J3 Micro_SD_Card_Det, J4 Conn_Coaxial, J5 Conn_Coaxial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

Commit message: update cause why not
Parts:
- removed the G*** at (231.2, 39.0)
- moved TP13 91.7 mm to (113.4, 91.3)
- moved TP12 85.5 mm to (115.5, 91.3)
- moved G*** 65.6 mm to (182.0, 55.5)
- moved U11 56.8 mm to (111.7, 100.8), turned to 180 degrees
- moved C12 48.8 mm to (100.8, 85.4)
- moved C28 48.5 mm to (100.9, 101.9), turned to 180 degrees
- moved C13 47.3 mm to (100.8, 82.4), turned to 90 degrees
- moved J4 46.4 mm to (115.8, 86.4), turned to 180 degrees
- moved C29 44.9 mm to (100.9, 100.4), turned to 180 degrees
- moved R25 44.9 mm to (114.7, 81.5), turned to 90 degrees
- moved C4 44.8 mm to (120.2, 86.0), turned to 270 degrees
- moved C14 43.7 mm to (12.7, 73.6)
- moved C17 43.7 mm to (17.3, 73.6)
- moved C20 43.7 mm to (18.8, 73.7)
- moved C21 43.7 mm to (20.3, 73.7)
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Routing:
- net /RADIO_RX: track 38.9 -> 5.20 mm
- net Net-(C3-Pad1): track 32.7 -> 2.37 mm
- net /RADIO_TX: track 35.5 -> 5.53 mm
- net +3V3: track 81.1 -> 55.4 mm
- net /nukes/External_Supply: track 75.2 -> 51.3 mm
- net /SCL: track 39.9 -> 18.1 mm, vias 0 -> 1
- net /CAN_RX: track 6.10 -> 25.7 mm, vias 0 -> 2
- net /usb-c/usb_D+: track 0.00 -> 15.6 mm, vias 0 -> 1
- net /GPS/TXD: track 0.00 -> 14.9 mm
- net Net-(J5-Pad1): track 0.00 -> 14.4 mm
- net GND: track 101.9 -> 116.1 mm
- net Net-(J11-Pad1): track 17.5 -> 3.83 mm
- net /GPS/RXD: track 0.00 -> 13.0 mm
- net Net-(D15-Pad2): track 30.2 -> 17.3 mm
- net /SDA: track 30.7 -> 18.7 mm
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Other:
- board text added: "ogres are like onions"
- board text removed: "to the moon"
