File: Bluetooth_Igniter/Bluetooth_ignite_receiver.sch (KiCad schematic (older format))
At the start: 28 parts, among them Q1 MMDT2222A, Q2 MMDT2222A, SW1 SW_Push, SW2 SW_Push, U1 CP2102N-A01-GQFN24, U2 ESP32-WROOM-32

Commit message: pcb routing
Parts:
- removed SW1, SW2: SW_Push, Button_Switch_SMD:SW_Push_1P1T_NO_CK_KMR2, symbol Switch:SW_Push
- added J6, J7: Conn_01x02_Male, Connector_PinHeader_2.54mm:PinHeader_1x02_P2.54mm_Vertical, symbol Connector:Conn_01x02_Male
- added TP? (x5): TestPoint, symbol Connector:TestPoint
Other:
- moved on the sheet: Q1A, Q2A, R1, R2
