File: Bluetooth_Igniter/pyros.sch (KiCad schematic (older format))
At the start: 21 parts, among them J1 Screw_Terminal_01x02, J2 Screw_Terminal_01x02, J3 Screw_Terminal_01x02, Q3 Q_NMOS_GSD, Q4 Q_NMOS_GSD, U3 LTV-817S, U4 LTV-817S

Commit message: pcb routing
Parts:
- J1, J2, J3: footprint iclrhw:PHOENIX_1757242 -> TerminalBlock_Phoenix:TerminalBlock_Phoenix_PT-1,5-2-5.0-H_1x02_P5.00mm_Horizontal
Changed lines of the file:
@@
 F 0 "J1" V 2772 3630 50  0000 L CNN
 F 1 "Screw_Terminal_01x02" V 2863 3630 50  0000 L CNN
-F 2 "iclrhw:PHOENIX_1757242" H 2900 3550 50  0001 C CNN
+F 2 "TerminalBlock_Phoenix:TerminalBlock_Phoenix_PT-1,5-2-5.0-H_1x02_P5.00mm_Horizontal" H 2900 3550 50  0001 C CNN
 F 3 "~" H 2900 3550 50  0001 C CNN
 	1    2900 3550
@@
 F 0 "J3" V 7422 3680 50  0000 L CNN
 F 1 "Screw_Terminal_01x02" V 7513 3680 50  0000 L CNN
-F 2 "iclrhw:PHOENIX_1757242" H 7550 3600 50  0001 C CNN
+F 2 "TerminalBlock_Phoenix:TerminalBlock_Phoenix_PT-1,5-2-5.0-H_1x02_P5.00mm_Horizontal" H 7550 3600 50  0001 C CNN
 F 3 "~" H 7550 3600 50  0001 C CNN
 	1    7550 3600
@@
 F 0 "J2" H 3480 1692 50  0000 L CNN
 F 1 "Screw_Terminal_01x02" H 3480 1601 50  0000 L CNN
-F 2 "iclrhw:PHOENIX_1757242" H 3400 1700 50  0001 C CNN
+F 2 "TerminalBlock_Phoenix:TerminalBlock_Phoenix_PT-1,5-2-5.0-H_1x02_P5.00mm_Horizontal" H 3400 1700 50  0001 C CNN
 F 3 "~" H 3400 1700 50  0001 C CNN
 	1    3400 1700
@@
 	2250 1700 3200 1700
 $Comp
-L power:GND #PWR?
+L power:GND #PWR0101
 U 1 1 60A35AE3
 P 2250 1800
-F 0 "#PWR?" H 2250 1550 50  0001 C CNN
+F 0 "#PWR0101" H 2250 1550 50  0001 C CNN
 F 1 "GND" H 2255 1627 50  0000 C CNN
 F 2 "" H 2250 1800 50  0001 C CNN
