File: Bluetooth_Igniter/Bluetooth_ignite_receiver.kicad_pcb (KiCad board)
At the start: 2 copper layers, 69 parts, among them J1 Screw_Terminal_01x02, J2 Screw_Terminal_01x02, J3 Screw_Terminal_01x02, J4 Screw_Terminal_01x02, J5 USB_C_Receptacle_USB2.0, Q1 MMDT2222A, Q2 MMDT2222A, Q3 Q_NMOS_GSD, Q4 Q_NMOS_GSD, SW1 SW_Push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

Commit message: pcb routing
Parts:
- removed SW1, SW2: SW_Push, Button_Switch_SMD:SW_Push_1P1T_NO_CK_KMR2
- added J6: Conn_01x02_Male, Connector_PinHeader_2.54mm:PinHeader_1x02_P2.54mm_Vertical, F.Cu at (32.7, 115.3)
- added J7: Conn_01x02_Male, Connector_PinHeader_2.54mm:PinHeader_1x02_P2.54mm_Vertical, F.Cu at (33.2, 89.8)
- J1, J2, J3, J4: footprint iclrhw:PHOENIX_1757242 -> TerminalBlock_Phoenix:TerminalBlock_Phoenix_PT-1,5-2-5.0-H_1x02_P5.00mm_Horizontal
- moved J1 9.25 mm to (66.4, 125.7), turned to 0 degrees
- moved J2 7.20 mm to (68.5, 86.9), turned to 180 degrees
- moved D10 6.24 mm to (75.0, 100.8)
- moved D11 6.24 mm to (73.4, 91.6)
- moved J5 6.24 mm to (68.6, 96.9)
- moved R22 6.24 mm to (74.9, 97.5)
- moved R23 6.24 mm to (74.9, 94.2)
- moved J3 5.97 mm to (54.6, 125.6), turned to 0 degrees
- moved REF** 5.26 mm to (81.9, 86.7)
- moved J4 3.81 mm to (57.3, 86.9), turned to 180 degrees
- moved REF** 2.86 mm to (32.2, 126.0)
- moved C8 2.42 mm to (58.0, 100.5)
- moved R3 1.81 mm to (70.8, 108.5)
- moved R5 1.75 mm to (71.2, 103.4), turned to 180 degrees
- moved D2 1.41 mm to (61.3, 104.3), turned to 180 degrees
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Routing:
- net /Cont1: track 2.77 -> 63.7 mm, vias 0 -> 2
- net /Nuke1: track 0.00 -> 50.3 mm, vias 0 -> 2
- net /pyros/Ext_supply: track 0.00 -> 43.8 mm
- net /BOOT: track 0.00 -> 37.2 mm, vias 0 -> 4
- net /Cont2: track 2.96 -> 38.0 mm, vias 0 -> 2
- net /usb/D+: track 8.08 -> 39.9 mm, vias 0 -> 4
- net /TXD: track 0.00 -> 30.5 mm, vias 0 -> 2
- net /EN: track 15.1 -> 45.6 mm
- net /RXD: track 0.00 -> 29.3 mm, vias 0 -> 2
- net /Nuke2: track 0.00 -> 26.8 mm, vias 0 -> 2
- net Net-(R24-Pad1): track 0.00 -> 24.6 mm
- net /RTS: track 4.50 -> 27.7 mm, vias 0 -> 2
- net /usb/VBUS: track 5.27 -> 28.3 mm, vias 0 -> 4
- net /PG: track 2.46 -> 21.0 mm
- net Net-(D5-Pad2): track 10.7 -> 27.2 mm
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Other:
- board outline added: 61.1 x 50.4 mm

Commit message: need to make pcb thinner
Routing:
- net /pyros/Ext_supply: track 43.8 -> 121.9 mm
- net +3V3: track 12.5 -> 20.7 mm, vias 0 -> 2
- net VDD: track 13.9 -> 17.0 mm
- added copper zone on B.Cu, net +3V3
- added copper zone on F.Cu, net GND
Changed lines of the file:
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@@
     (thickness 1.6)
     (drawings 6)
-    (tracks 457)
+    (tracks 476)
     (zones 0)
     (modules 69)
@@
   )
   (setup
-    (last_trace_width 1)
-    (user_trace_width 1)
+    (last_trace_width 0.25)
+    (user_trace_width 0.4)
     (trace_clearance 0.2)
-    (zone_clearance 0.508)
+    (zone_clearance 0.2)
     (zone_45_only no)
     (trace_min 0.2)
@@
   (segment (start 57.4421 93.8019) (end 58.24251 93.00149) (width 0.25) (layer F.Cu) (net 2))
   (segment (start 29.845 110.1) (end 29.845 110.865002) (width 0.25) (layer F.Cu) (net 2))
+  (segment (start 41.1991 112.4585) (end 41.4401 112.4585) (width 0.25) (layer F.Cu) (net 2))
+  (via (at 42.5958 113.6142) (size 0.8) (drill 0.4) (layers F.Cu B.Cu) (net 2))
+  (segment (start 41.4401 112.4585) (end 42.5958 113.6142) (width 0.25) (layer F.Cu) (net 2))
+  (segment (start 71.9831 103.4034) (end 74.6379 103.4034) (width 0.25) (layer F.Cu) (net 2))
+  (via (at 77.2033 105.9688) (size 0.8) (drill 0.4) (layers F.Cu B.Cu) (net 2))
+  (segment (start 74.6379 103.4034) (end 77.2033 105.9688) (width 0.25) (layer F.Cu) (net 2))
   (segment (start 39.5468 116.0775) (end 37.8968 114.4275) (width 0.25) (layer F.Cu) (net 3))
   (segment (start 39.5478 116.0775) (end 39.5468 116.0775) (width 0.25) (layer F.Cu) (net 3))
@@
   (segment (start 50.7619 88.4339) (end 50.7619 96.3673) (width 1) (layer F.Cu) (net 6))
   (segment (start 50.7619 96.3673) (end 50.7619 96.532102) (width 0.25) (layer F.Cu) (net 6))
+  (segment (start 52.021699 97.926901) (end 52.7667 97.926901) (width 0.4) (layer F.Cu) (net 6))
+  (segment (start 51.941699 97.846901) (end 52.021699 97.926901) (width 0.4) (layer F.Cu) (net 6))
+  (segment (start 51.941699 97.072099) (end 51.941699 97.846901) (width 0.4) (layer F.Cu) (net 6))
+  (segment (start 51.2369 96.3673) (end 51.941699 97.072099) (width 0.4) (layer F.Cu) (net 6))
+  (segment (start 50.7619 96.3673) (end 51.2369 96.3673) (width 0.4) (layer F.Cu) (net 6))
   (segment (start 56.8249 100.4951) (end 55.7167 99.3869) (width 0.25) (layer F.Cu) (net 7))
   (segment (start 57.2383 100.4951) (end 56.8249 100.4951) (width 0.25) (layer F.Cu) (net 7))
@@
   (segment (start 32.7792 112.4839) (end 32.02919 113.23391) (width 0.25) (layer F.Cu) (net 12))
   (segment (start 62.680589 87.805511) (end 63.5419 86.9442) (width 0.25) (layer F.Cu) (net 13))
-  (segment (start 57.635399 127.577601) (end 59.6354 125.5776) (width 1) (layer F.Cu) (net 13))
-  (segment (start 52.775399 127.577601) (end 57.635399 127.577601) (width 1) (layer F.Cu) (net 13))
-  (segment (start 51.994591 126.796793) (end 52.775399 127.577601) (width 1) (layer F.Cu) (net 13))
-  (segment (start 52.8196 117.1702) (end 51.994591 117.995209) (width 1) (layer F.Cu) (net 13))
   (segment (start 71.4083 118.8986) (end 71.4083 125.73) (width 1) (layer F.Cu) (net 13))
   (segment (start 73.4161 116.8908) (end 71.4083 118.8986) (width 1) (layer F.Cu) (net 13))
@@
   (segment (start 61.787801 127.730001) (end 59.6354 125.5776) (width 1) (layer F.Cu) (net 13))
   (segment (start 71.4083 125.73) (end 69.408299 127.730001) (width 1) (layer F.Cu) (net 13))
+  (segment (start 52.8196 117.1702) (end 51.994591 117.995209) (width 1) (layer F.Cu) (net 13))
   (segment (start 51.994591 117.995209) (end 51.994591 126.796793) (width 1) (layer F.Cu) (net 13))
+  (segment (start 51.994591 126.796793) (end 52.775399 127.577601) (width 1) (layer F.Cu) (net 13))
+  (segment (start 52.775399 127.577601) (end 57.635399 127.577601) (width 1) (layer F.Cu) (net 13))
+  (segment (start 57.635399 127.577601) (end 59.6354 125.5776) (width 1) (layer F.Cu) (net 13))
+  (segment (start 63.5419 86.9442) (end 61.541899 84.944199) (width 1) (layer B.Cu) (net 13))
+  (segment (start 36.94362 109.869422) (end 43.927222 109.869422) (width 1) (layer B.Cu) (net 13))
+  (segment (start 61.541899 84.944199) (end 47.196899 84.944199) (width 1) (layer B.Cu) (net 13))
+  (segment (start 47.196899 84.944199) (end 33.799599 98.341499) (width 1) (layer B.Cu) (net 13))
+  (segment (start 33.799599 98.341499) (end 33.799599 106.725401) (width 1) (layer B.Cu) (net 13))
+  (segment (start 33.799599 106.725401) (end 36.94362 109.869422) (width 1) (layer B.Cu) (net 13))
+  (segment (start 43.927222 109.869422) (end 59.6354 125.5776) (width 1) (layer B.Cu) (net 13))
   (segment (start 74.0286 118.4658) (end 73.9526 118.5418) (width 0.25) (layer F.Cu) (net 14))
   (segment (start 75.6036 116.8908) (end 73.9526 118.5418) (width 0.25) (layer F.Cu) (net 14))
@@
   (segment (start 70.0151 108.4077) (end 69.9648 108.458) (width 0.25) (layer F.Cu) (net 37))
   (segment (start 70.0151 107.315) (end 70.0151 108.4077) (width 0.25) (layer F.Cu) (net 37))
-  (segment (start 65.8363 108.7242) (end 66.6496 109.5375) (width 0.25) (layer F.Cu) (net 37))
   (segment (start 65.8363 108.4072) (end 65.8363 108.7242) (width 0.25) (layer F.Cu) (net 37))
-  (segment (start 69.71189 109.5375) (end 66.6496 109.5375) (width 0.25) (layer F.Cu) (net 37))
+  (segment (start 69.341399 109.081401) (end 69.9648 108.458) (width 0.25) (layer F.Cu) (net 37))
+  (segment (start 66.510501 109.081401) (end 69.341399 109.081401) (width 0.25) (layer F.Cu) (net 37))
+  (segment (start 65.8363 108.4072) (end 66.510501 109.081401) (width 0.25) (layer F.Cu) (net 37))
   (segment (start 70.3331 104.311022) (end 70.3331 103.4034) (width 0.25) (layer F.Cu) (net 38))
   (segment (start 69.403222 105.2409) (end 70.3331 104.311022) (width 0.25) (layer F.Cu) (net 38))
@@
   (segment (start 37.15329 90.340632) (end 37.463622 90.0303) (width 0.25) (layer F.Cu) (net 86))
   (segment (start 32.385 93.1) (end 32.385 91.85) (width 0.25) (layer F.Cu) (net 86))
+  (zone (net 1) (net_name GND) (layer F.Cu) (hatch edge 0.508)
+    (connect_pads (clearance 0.2))
+    (min_thickness 0.254)
+    (fill yes (arc_segments 32) (thermal_gap 0.508) (thermal_bridge_width 0.508))
+    (polygon
+      (pts
+        (xy 89.8017 80.6704) (xy 90.2462 132.6007) (xy 25.5397 132.7785) (xy 25.8064 80.6069)
+      )
+    )
+  )
+  (zone (net 2) (net_name +3V3) (layer B.Cu) (hatch edge 0.508)
+    (connect_pads (clearance 0.4))
+    (min_thickness 0.254)
+    (fill yes (arc_segments 32) (thermal_gap 0.508) (thermal_bridge_width 0.508))
+    (polygon
+      (pts
+        (xy 91.1225 132.8928) (xy 24.5364 133.8072) (xy 25.1841 80.2005) (xy 91.2495 79.5528)
+      )
+    )
+  )
 )
