File: PickleRick/_autosave-PickleRick.kicad_pcb (KiCad board)
At the start: 4 copper layers, 100 x 37 mm, 176 parts, among them J1 Conn_01x06_Male, J10 Conn_01x03_Male, J11 Conn_01x02_Male, J12 Conn_01x05_Male, J14 DeployLipo, J15 UCLipo, J16 Conn_Coaxial, J17 USB_C_Receptacle_USB2.0, J18 Conn_Coaxial, J2 Conn_01x02_Male, J3 Conn_01x02_Male, J4 Micro_SD_Card_Det, J5 CON7_1X7_DRH_HPI125_TYC, J6 Screw_Terminal_01x08, Q1 MMDT2222A, Q10 AO3401A, Q2 PMV20ENR, Q3 NCV8415STT1G, Q4 NCV8415STT1G, Q5 NCV8415STT1G, Q6 NCV8415STT1G, Q7 SI4143DY-T1-GE3, Q8 SI4143DY-T1-GE3, Q9 AO3401A, U1 SN65HVD230, U10 LTC4411ES5TRMPBF, U11 LTC4411ES5TRMPBF, U12 LT1963AxST-3.3, U13 LTC4412xS6, U14 LTC4412xS6, U15 LTC4412xS6, U16 LTC4412xS6, U17 MAX-M8Q, U18 CP2102-GMR-QFN28, U19 RFM95W-868S2, U2 ESP32-WROOM-32D, U3 MS5607-02BA, U4 LTV-247, U5 PCA9534RGVR, U6 PCA9685BS, U7 H3LIS100DLTR, U8 ICM-20608-G, U9 MMC5983MA

Commit message: pickle ready for review
Parts:
- moved REF** 43.6 mm to (147.9, 79.0), turned to 180 degrees
- moved G*** 1.93 mm to (167.2, 79.7), turned to -90 degrees
Other:
- board text added: "NUKES"
- board text removed: "PYROS"
Changed lines of the file:
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@@
   )
   (footprint "iclr:Write_Pad" (layer "F.Cu")
-    (at 191.575 77.875)
+    (at 147.95 78.975 180)
     (attr through_hole)
     (fp_text reference "REF**" (at 0 5.88) (layer "F.SilkS") hide
@@
   )
   (footprint "iclr:pickle_ric" (layer "B.Cu")
-    (at 167.73 77.84 90)
+    (at 167.2 79.7 -90)
     (attr through_hole)
     (fp_text reference "G***" (at 0 0 90) (layer "B.SilkS") hide
@@
     (pad "8" smd rect (at -3.500999 4.9784) (size 2.413 3.302) (layers "B.Cu" "B.Paste" "B.Mask"))
     (pad "9" smd rect (at 12.501001 4.9784) (size 2.413 3.302) (layers "B.Cu" "B.Paste" "B.Mask"))
+    (model "/Users/kiran/Documents/Projects/ICLR/iclr-hw/3d/c-292227-7-a1-3d.stp"
+      (offset (xyz 4.5 8.5 2.5))
+      (scale (xyz 1 1 1))
+      (rotate (xyz -90 0 180))
+    )
   )
   (footprint "Jumper:SolderJumper-2_P1.3mm_Open_RoundedPad1.0x1.5mm" (layer "B.Cu")
@@
   (gr_line (start 214 78.5) (end 99.5 78.5) (layer "User.1") (width 0.15))
   (gr_line (start 214 97) (end 214 78.5) (layer "User.1") (width 0.15))
-  (gr_text "D-" (at 163.425 87.525) (layer "B.SilkS")
+  (gr_text "D-" (at 163.425 87.525 180) (layer "B.SilkS")
     (effects (font (size 1 1) (thickness 0.15)) (justify mirror))
   )
-  (gr_text "D+" (at 161.325 87.6) (layer "B.SilkS")
+  (gr_text "D+" (at 161.325 87.6 180) (layer "B.SilkS")
     (effects (font (size 1 1) (thickness 0.15)) (justify mirror))
   )
@@
     (effects (font (size 1 1) (thickness 0.15)) (justify mirror))
   )
-  (gr_text "Designed By Kiran de Silva\nElectronics & Payload 2022" (at 149.25 78.4 270) (layer "B.SilkS")
+  (gr_text "Designed By Kiran de Silva\nElectronics & Payload 2022" (at 195.5 78.175 90) (layer "B.SilkS")
     (effects (font (size 1 1) (thickness 0.15)) (justify mirror))
   )
@@
     (effects (font (size 1 1) (thickness 0.15)))
   )
-  (gr_text "PYROS" (at 128.075 66.325 180) (layer "F.SilkS")
+  (gr_text "NUKES" (at 128.075 66.325 180) (layer "F.SilkS")
     (effects (font (size 1 1) (thickness 0.15)))
   )
