File: PickleRick/IMU.kicad_sch (KiCad schematic)
At the start: 11 parts, among them U7 H3LIS100DLTR, U8 ICM-20608-G, U9 MMC5983MA

Commit message: switched vspi and hspi labels so they are consistent with documentation
Parts:
- U7: value H3LIS100DLTR -> H3LIS331DLTR
Changed lines of the file:
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@@
     (in_bom yes) (on_board yes) (fields_autoplaced)
     (property "Reference" "U7" (id 0) (at 65.405 40.64 0))
-    (property "Value" "H3LIS100DLTR" (id 1) (at 65.405 43.18 0))
+    (property "Value" "H3LIS331DLTR" (id 1) (at 65.405 43.18 0))
     (property "Footprint" "iclr:PQFN50P300X300X100-16N" (id 2) (at 65.405 58.42 0)
       (effects (font (size 1.27 1.27)) (justify left bottom) hide)
