File: PickleRick/PickleRick.kicad_sch (KiCad schematic)
At the start: 73 parts, among them J1 Conn_01x05_Male, J2 Conn_01x02_Male, J3 Conn_01x02_Male, J4 Micro_SD_Card_Det, J5 Conn_01x07_Male, Q1 MMDT2222A, Q2 PMV20ENR, U1 SN65HVD230, U2 ESP32-WROOM-32D, U3 MS5607-02BA

Commit message: first full layout of pickle complete
Parts:
- removed BZ1: Buzzer, Buzzer_Beeper:Buzzer_TDK_PS1240P02BT_D12.2mm_H6.5mm, symbol Device:Buzzer
- removed J1: Conn_01x05_Male, Connector_PinSocket_2.54mm:PinSocket_1x05_P2.54mm_Vertical, symbol Connector:Conn_01x05_Male
- removed TP1, TP10, TP2, TP4, TP7, TP9: TestPoint, TestPoint:TestPoint_THTPad_1.0x1.0mm_Drill0.5mm, symbol Connector:TestPoint
- added C23, C36: 10uF, Capacitor_SMD:C_0603_1608Metric, symbol Device:C_Small
- added C27: 160pF, Capacitor_SMD:C_0603_1608Metric, symbol Device:C_Small
- added C28: 100nF, Capacitor_SMD:C_0603_1608Metric, symbol Device:C_Small
- added C37: 0.1uF, Capacitor_SMD:C_0603_1608Metric, symbol Device:C
- added C38: 220pF, Capacitor_SMD:C_0603_1608Metric, symbol Device:C_Small
- added C39: 220 pF, Capacitor_SMD:C_0603_1608Metric, symbol Device:C_Small
- added D19: SM712_SOT23, Package_TO_SOT_SMD:SOT-23, symbol Diode:SM712_SOT23
- added J1: Conn_01x06_Male, Connector_Molex:Molex_Mini-Fit_Jr_5566-06A_2x03_P4.20mm_Vertical, symbol Connector:Conn_01x06_Male
- added J10: Conn_01x03_Male, Connector_PinHeader_2.54mm:PinHeader_1x03_P2.54mm_Vertical, symbol Connector:Conn_01x03_Male
- added J11: Conn_01x02_Male, Connector_JST:JST_PH_B2B-PH-K_1x02_P2.00mm_Vertical, symbol Connector:Conn_01x02_Male
- added JP1: SolderJumper_2_Open, Jumper:SolderJumper-2_P1.3mm_Open_RoundedPad1.0x1.5mm, symbol Jumper:SolderJumper_2_Open
- added R39, R40: 90, Resistor_SMD:R_0603_1608Metric, symbol Device:R_Small
- added R41: 10k, Resistor_SMD:R_0603_1608Metric, symbol Device:R_Small
- added R48, R49: 60, Resistor_SMD:R_0603_1608Metric, symbol Device:R
- TP11, TP12, TP13, TP14, TP15, TP16, TP17, TP18, TP19, TP20, TP21, TP22, TP23, TP24, TP25, TP26, TP27, TP28, TP3, TP5, TP6, TP8: footprint TestPoint:TestPoint_THTPad_1.0x1.0mm_Drill0.5mm -> TestPoint:TestPoint_Pad_D1.0mm
Connections:
- net +3V3: now also C23.1, C28.1, C36.1, J11.2 (Pin_2)
- net BARO_CS: now also U2.24 (IO2); no longer U2.12 (IO27)
- net Buzzer: now also U2.12 (IO27); no longer U2.24 (IO2)
- net CAN_HIGH: now also C38.2, D19.2 (A2), J1.5 (Pin_5), R48.1
- net CAN_LOW: now also C39.2, D19.1 (A1), J1.6 (Pin_6), R49.2
- net CAN_RX: now also R40.1; no longer U1.4 (R)
- net CAN_TX: now also R39.1; no longer U1.1 (D)
- net GND: now also C23.2, C27.1, C28.2, C36.2, C37.2, C38.1, C39.1, D19.3 (common), J1.1 (Pin_1), J1.2 (Pin_2), J10.1 (Pin_1), R41.2; no longer U1.8 (Rs)
- net HSPI_MISO: now also TP18.1, U2.31 (IO19); no longer TP11.1, U2.14 (IO12)
- net HSPI_MOSI: now also TP19.1, U2.37 (IO23); no longer TP12.1, U2.16 (IO13)
- net HSPI_SCLK: now also TP17.1, U2.30 (IO18); no longer TP13.1, U2.13 (IO14)
- net SCL: now also J10.2 (Pin_2)
- net SDA: now also J10.3 (Pin_3)
- net VSPI_MISO: now also TP11.1, U2.14 (IO12); no longer TP18.1, U2.31 (IO19)
- net VSPI_MOSI: now also TP12.1, U2.16 (IO13); no longer TP19.1, U2.37 (IO23)
- net VSPI_SCLK: now also TP13.1, U2.13 (IO14); no longer TP17.1, U2.30 (IO18)
- net power/RBUS_24V_IN: now also J1.4 (Pin_4)
- net power/RBUS_3.3_IN: now also J1.3 (Pin_3)
- net at D6.2 (A): now also J11.1 (Pin_1)
- net Vref: now reaches U1.5 (Vref)
- net Vref: now also JP1.1 (A)
- new net: C37.1, JP1.2 (B), R48.2, R49.1
- new net: R41.1, U1.8 (Rs)
- new net: C27.2, R39.2, U1.1 (D)
- new net: R40.2, U1.4 (R)
- no-connect marks 9 -> 8
Other:
- moved on the sheet: C6, D1, D2, D3, D4, D5, R10, R11, R7, R8, R9, TP22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

Commit message: pickle layed out
Connections:
- net SCL: now also J10.3 (Pin_3); no longer J10.2 (Pin_2)
- net SDA: now also J10.2 (Pin_2); no longer J10.3 (Pin_3)
Other:
- moved on the sheet: J10
Changed lines of the file:
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@@
   (junction (at 86.995 83.82) (diameter 0) (color 0 0 0 0)
   )
+  (junction (at 147.32 139.7) (diameter 0) (color 0 0 0 0)
+  )
   (junction (at 82.55 74.93) (diameter 0) (color 0 0 0 0)
   )
@@
   (junction (at 153.67 30.48) (diameter 0) (color 0 0 0 0)
   )
-  (junction (at 147.32 139.7) (diameter 0) (color 0 0 0 0)
-  )
   (junction (at 125.73 24.13) (diameter 0) (color 0 0 0 0)
   )
+  (junction (at 144.78 137.16) (diameter 0) (color 0 0 0 0)
+  )
   (junction (at 146.05 129.54) (diameter 0) (color 0 0 0 0)
   )
@@
   (junction (at 121.92 33.02) (diameter 0) (color 0 0 0 0)
   )
-  (junction (at 144.78 137.16) (diameter 0) (color 0 0 0 0)
-  )
   (junction (at 74.93 66.04) (diameter 0) (color 0 0 0 0)
   )
@@
     (stroke (width 0) (type default) (color 0 0 0 0))
   )
-  (wire (pts (xy 110.49 137.16) (xy 144.78 137.16))
-    (stroke (width 0) (type default) (color 0 0 0 0))
-  )
   (wire (pts (xy 34.29 137.16) (xy 30.48 137.16))
     (stroke (width 0) (type default) (color 0 0 0 0))
@@
     (stroke (width 0) (type default) (color 0 0 0 0))
   )
+  (wire (pts (xy 110.49 137.16) (xy 144.78 137.16))
+    (stroke (width 0) (type default) (color 0 0 0 0))
+  )
   (wire (pts (xy 57.15 170.18) (xy 63.5 170.18))
     (stroke (width 0) (type default) (color 0 0 0 0))
@@
     (stroke (width 0) (type default) (color 0 0 0 0))
   )
+  (wire (pts (xy 144.78 137.16) (xy 160.02 137.16))
+    (stroke (width 0) (type default) (color 0 0 0 0))
+  )
   (wire (pts (xy 267.97 147.32) (xy 260.35 147.32))
     (stroke (width 0) (type default) (color 0 0 0 0))
@@
     (stroke (width 0) (type default) (color 0 0 0 0))
   )
-  (wire (pts (xy 144.78 137.16) (xy 157.48 137.16))
-    (stroke (width 0) (type default) (color 0 0 0 0))
-  )
   (wire (pts (xy 125.73 24.13) (xy 130.81 24.13))
     (stroke (width 0) (type default) (color 0 0 0 0))
@@
     (stroke (width 0) (type default) (color 0 0 0 0))
   )
-  (wire (pts (xy 147.32 139.7) (xy 147.32 134.62))
+  (wire (pts (xy 147.32 134.62) (xy 147.32 139.7))
     (stroke (width 0) (type default) (color 0 0 0 0))
   )
@@
     (stroke (width 0) (type default) (color 0 0 0 0))
   )
-  (wire (pts (xy 160.02 139.7) (xy 160.02 137.16))
-    (stroke (width 0) (type default) (color 0 0 0 0))
-  )
   (wire (pts (xy 41.91 157.48) (xy 53.34 157.48))
     (stroke (width 0) (type default) (color 0 0 0 0))
@@
     (stroke (width 0) (type default) (color 0 0 0 0))
   )
+  (wire (pts (xy 160.02 137.16) (xy 160.02 135.89))
+    (stroke (width 0) (type default) (color 0 0 0 0))
+  )
   (wire (pts (xy 35.56 90.17) (xy 41.91 90.17))
     (stroke (width 0) (type default) (color 0 0 0 0))
@@
     (stroke (width 0) (type default) (color 0 0 0 0))
   )
-  (wire (pts (xy 147.32 139.7) (xy 160.02 139.7))
-    (stroke (width 0) (type default) (color 0 0 0 0))
-  )
   (wire (pts (xy 84.455 91.44) (xy 86.995 91.44))
     (stroke (width 0) (type default) (color 0 0 0 0))
@@
     (stroke (width 0) (type default) (color 0 0 0 0))
   )
+  (wire (pts (xy 147.32 139.7) (xy 157.48 139.7))
+    (stroke (width 0) (type default) (color 0 0 0 0))
+  )
   (wire (pts (xy 223.52 149.86) (xy 233.68 149.86))
     (stroke (width 0) (type default) (color 0 0 0 0))
@@
     (stroke (width 0) (type default) (color 0 0 0 0))
   )
+  (wire (pts (xy 157.48 135.89) (xy 157.48 139.7))
+    (stroke (width 0) (type default) (color 0 0 0 0))
+  )
   (wire (pts (xy 121.92 24.13) (xy 121.92 33.02))
     (stroke (width 0) (type default) (color 0 0 0 0))
@@
     (effects (font (size 1.27 1.27)) (justify left bottom))
   )
-  (symbol (lib_id "power:GND") (at 162.56 137.16 0) (unit 1)
+  (symbol (lib_id "power:GND") (at 162.56 135.89 0) (unit 1)
     (in_bom yes) (on_board yes)
-    (property "Reference" "#PWR034" (id 0) (at 162.56 143.51 0)
+    (property "Reference" "#PWR034" (id 0) (at 162.56 142.24 0)
       (effects (font (size 1.27 1.27)) hide)
     )
-    (property "Value" "GND" (id 1) (at 162.56 140.97 0))
-    (property "Footprint" "" (id 2) (at 162.56 137.16 0)
+    (property "Value" "GND" (id 1) (at 162.56 139.7 0))
+    (property "Footprint" "" (id 2) (at 162.56 135.89 0)
       (effects (font (size 1.27 1.27)) hide)
     )
-    (property "Datasheet" "" (id 3) (at 162.56 137.16 0)
+    (property "Datasheet" "" (id 3) (at 162.56 135.89 0)
       (effects (font (size 1.27 1.27)) hide)
     )
@@
     (pin "2")
   )
-  (symbol (lib_id "Connector:Conn_01x03_Male") (at 160.02 132.08 270) (unit 1)
+  (symbol (lib_id "Connector:Conn_01x03_Male") (at 160.02 130.81 270) (unit 1)
     (in_bom yes) (on_board yes) (fields_autoplaced)
-    (property "Reference" "J10" (id 0) (at 160.02 127 90))
-    (property "Value" "Conn_01x03_Male" (id 1) (at 160.02 129.54 90))
-    (property "Footprint" "Connector_PinHeader_2.54mm:PinHeader_1x03_P2.54mm_Vertical" (id 2) (at 160.02 132.08 0)
+    (property "Reference" "J10" (id 0) (at 160.02 125.73 90))
+    (property "Value" "Conn_01x03_Male" (id 1) (at 160.02 128.27 90))
+    (property "Footprint" "Connector_PinHeader_2.54mm:PinHeader_1x03_P2.54mm_Vertical" (id 2) (at 160.02 130.81 0)
       (effects (font (size 1.27 1.27)) hide)
     )
-    (property "Datasheet" "~" (id 3) (at 160.02 132.08 0)
+    (property "Datasheet" "~" (id 3) (at 160.02 130.81 0)
       (effects (font (size 1.27 1.27)) hide)
     )
@@
       (reference "#PWR038") (unit 1) (value "GND") (footprint "")
     )
-    (path "/ca0eab8e-e3fd-464d-bb03-d1603b8a651b/fa24134d-d746-49ac-8434-03d3cb51b93d"
-      (reference "#PWR039") (unit 1) (value "GND") (footprint "")
-    )
     (path "/ca0eab8e-e3fd-464d-bb03-d1603b8a651b/95fdd41f-879b-4183-897c-ad6f1e5df1b2"
       (reference "#PWR040") (unit 1) (value "+24V") (footprint "")
     )
-    (path "/ca0eab8e-e3fd-464d-bb03-d1603b8a651b/851f889c-76e5-4629-b1ed-c8947a5326da"
-      (reference "#PWR041") (unit 1) (value "GND") (footprint "")
-    )
     (path "/ca0eab8e-e3fd-464d-bb03-d1603b8a651b/eec6d8e9-9bf8-4a69-a5ed-df68bef09560"
       (reference "#PWR042") (unit 1) (value "+24V") (footprint "")
@@
       (reference "#PWR051") (unit 1) (value "GND") (footprint "")
     )
-    (path "/ca0eab8e-e3fd-464d-bb03-d1603b8a651b/448040ca-a02e-4b7e-8437-aed42d571bd5"
-      (reference "#PWR052") (unit 1) (value "GND") (footprint "")
-    )
-    (path "/ca0eab8e-e3fd-464d-bb03-d1603b8a651b/91e33441-2ea9-4180-a411-2942eb347cb7"
-      (reference "#PWR053") (unit 1) (value "GND") (footprint "")
-    )
     (path "/ca0eab8e-e3fd-464d-bb03-d1603b8a651b/4ff4deec-58c6-420b-b444-b84fc0a8e9e7"
       (reference "#PWR054") (unit 1) (value "GND") (footprint "")
@@
       (reference "D10") (unit 1) (value "D_Schottky") (footprint "Diode_SMD:D_SOD-128")
     )
-    (path "/ca0eab8e-e3fd-464d-bb03-d1603b8a651b/9931a64b-fd36-4110-8ce0-14e327e359d3"
-      (reference "D11") (unit 1) (value "CONTINUITY") (footprint "LED_SMD:LED_0603_1608Metric")
-    )
-    (path "/ca0eab8e-e3fd-464d-bb03-d1603b8a651b/5a90598c-3983-451b-a2d7-b73f587c4f67"
-      (reference "D12") (unit 1) (value "CONTINUITY") (footprint "LED_SMD:LED_0603_1608Metric")
-    )
     (path "/ca0eab8e-e3fd-464d-bb03-d1603b8a651b/8b7b86c2-493b-42f3-9e13-3f8dc5985623"
       (reference "D15") (unit 1) (value "D_Schottky") (footprint "Diode_SMD:D_SOD-128")
@@
       (reference "D16") (unit 1) (value "D_Schottky") (footprint "Diode_SMD:D_SOD-128")
     )
-    (path "/ca0eab8e-e3fd-464d-bb03-d1603b8a651b/35d7ebc4-2900-4bf5-b916-6d54f67d0fcf"
-      (reference "D17") (unit 1) (value "CONTINUITY") (footprint "LED_SMD:LED_0603_1608Metric")
-    )
-    (path "/ca0eab8e-e3fd-464d-bb03-d1603b8a651b/72c65652-f48a-44b8-a631-4aec028df1f9"
-      (reference "D18") (unit 1) (value "CONTINUITY") (footprint "LED_SMD:LED_0603_1608Metric")
-    )
     (path "/17915c67-0755-4b4b-9b9a-cfdcf9b1cb37"
       (reference "D19") (unit 1) (value "SM712_SOT23") (footprint "Package_TO_SOT_SMD:SOT-23")
@@
       (reference "R27") (unit 1) (value "1K") (footprint "Resistor_SMD:R_0603_1608Metric")
     )
-    (path "/ca0eab8e-e3fd-464d-bb03-d1603b8a651b/53c8e8c3-ce93-478f-8a85-d775e7b02cdd"
-      (reference "R28") (unit 1) (value "2K") (footprint "Resistor_SMD:R_0603_1608Metric")
-    )
     (path "/ca0eab8e-e3fd-464d-bb03-d1603b8a651b/d7977444-08fa-4843-83fb-a1317f1a30c1"
       (reference "R29") (unit 1) (value "1K") (footprint "Resistor_SMD:R_0603_1608Metric")
     )
-    (path "/ca0eab8e-e3fd-464d-bb03-d1603b8a651b/f6f3abb2-e5dd-46ed-ba63-e828a7cb795c"
-      (reference "R30") (unit 1) (value "2K") (footprint "Resistor_SMD:R_0603_1608Metric")
-    )
     (path "/ca0eab8e-e3fd-464d-bb03-d1603b8a651b/c4d9bc73-27a3-45e8-9f5d-4537c1fd0ae5"
       (reference "R33") (unit 1) (value "500") (footprint "Resistor_SMD:R_0603_1608Metric")
@@
       (reference "R36") (unit 1) (value "1K") (footprint "Resistor_SMD:R_0603_1608Metric")
     )
-    (path "/ca0eab8e-e3fd-464d-bb03-d1603b8a651b/09e25dcd-4ab0-4a31-828f-7d36c6ed6bc6"
-      (reference "R37") (unit 1) (value "2K") (footprint "Resistor_SMD:R_0603_1608Metric")
-    )
-    (path "/ca0eab8e-e3fd-464d-bb03-d1603b8a651b/5e3b5489-675b-461b-b0fd-9ce720cc17cb"
-      (reference "R38") (unit 1) (value "2K") (footprint "Resistor_SMD:R_0603_1608Metric")
-    )
     (path "/d633c156-e7cb-4efd-99b6-00516a628c16"

Commit message: pickle update
Parts:
- removed J5: Conn_01x07_Male, Connector_JST:JST_GH_SM07B-GHS-TB_1x07-1MP_P1.25mm_Horizontal, symbol Connector:Conn_01x07_Male
- removed TP5: TestPoint, TestPoint:TestPoint_Pad_D1.0mm, symbol Connector:TestPoint
- added J5: 292227-7, iclr:292227-7, symbol iclr:292227-7
- added TP1, TP2: TestPoint, TestPoint:TestPoint_Pad_D1.0mm, symbol Connector:TestPoint
Connections:
- net +3V3: now also J5.1
- net DTR: now also TP1.1
- net GND: now also J5.4
- net HSPI_MISO: now also J5.6
- net HSPI_MOSI: now also J5.3
- net HSPI_SCLK: now also J5.5
- net RTS: now also TP2.1
- net SD2_CS: now also J5.2
- net SD2_DET: now also J5.7
Other:
- sheet power ports: added UC_Lipo_Scaled; removed none
Changed lines of the file:
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@@
     (stroke (width 0) (type default) (color 0 0 0 0))
   )
+  (wire (pts (xy 59.69 33.02) (xy 68.58 33.02))
+    (stroke (width 0) (type default) (color 0 0 0 0))
+  )
   (wire (pts (xy 158.75 45.72) (xy 167.64 45.72))
     (stroke (width 0) (type default) (color 0 0 0 0))
@@
     (effects (font (size 1.27 1.27)) (justify left bottom))
   )
+  (label "BattVolt" (at 68.58 33.02 180)
+    (effects (font (size 1.27 1.27)) (justify right bottom))
+  )
   (symbol (lib_id "power:GND") (at 162.56 135.89 0) (unit 1)
     (in_bom yes) (on_board yes)
@@
     (pin "1")
   )
-  (symbol (lib_id "Connector:Conn_01x07_Male") (at 264.16 33.02 180) (unit 1)
-    (in_bom yes) (on_board yes) (fields_autoplaced)
-    (property "Reference" "J5" (id 0) (at 265.43 31.7499 0)
-      (effects (font (size 1.27 1.27)) (justify right))
-    )
-    (property "Value" "Conn_01x07_Male" (id 1) (at 265.43 34.2899 0)
-      (effects (font (size 1.27 1.27)) (justify right))
-    )
-    (property "Footprint" "Connector_JST:JST_GH_SM07B-GHS-TB_1x07-1MP_P1.25mm_Horizontal" (id 2) (at 264.16 33.02 0)
-      (effects (font (size 1.27 1.27)) hide)
-    )
-    (property "Datasheet" "~" (id 3) (at 264.16 33.02 0)
-      (effects (font (size 1.27 1.27)) hide)
-    )
-    (pin "1")
-    (pin "2")
-    (pin "3")
-    (pin "4")
-    (pin "5")
-    (pin "6")
-    (pin "7")
-  )
   (symbol (lib_id "Device:R_Small") (at 156.21 53.34 270) (unit 1)
     (in_bom yes) (on_board yes)
@@
     (pin "2")
   )
+  (symbol (lib_id "Connector:TestPoint") (at 20.32 151.13 90) (unit 1)
+    (in_bom yes) (on_board yes) (fields_autoplaced)
+    (property "Reference" "TP2" (id 0) (at 17.018 144.78 90))
+    (property "Value" "TestPoint" (id 1) (at 17.018 147.32 90))
+    (property "Footprint" "TestPoint:TestPoint_Pad_D1.0mm" (id 2) (at 20.32 146.05 0)
+      (effects (font (size 1.27 1.27)) hide)
+    )
+    (property "Datasheet" "~" (id 3) (at 20.32 146.05 0)
+      (effects (font (size 1.27 1.27)) hide)
+    )
+    (pin "1")
+  )
   (symbol (lib_id "Device:C_Small") (at 25.4 170.18 270) (unit 1)
     (in_bom yes) (on_board yes)
@@
     (pin "2")
   )
-  (symbol (lib_id "Connector:TestPoint") (at 124.46 101.6 270) (unit 1)
-    (in_bom yes) (on_board yes) (fields_autoplaced)
-    (property "Reference" "TP5" (id 0) (at 129.54 100.3299 90)
-      (effects (font (size 1.27 1.27)) (justify left))
-    )
-    (property "Value" "TestPoint" (id 1) (at 129.54 102.8699 90)
-      (effects (font (size 1.27 1.27)) (justify left))
-    )
-    (property "Footprint" "TestPoint:TestPoint_Pad_D1.0mm" (id 2) (at 124.46 106.68 0)
-      (effects (font (size 1.27 1.27)) hide)
-    )
-    (property "Datasheet" "~" (id 3) (at 124.46 106.68 0)
-      (effects (font (size 1.27 1.27)) hide)
-    )
-    (pin "1")
-  )
   (symbol (lib_id "power:GND") (at 45.72 171.45 0) (unit 1)
     (in_bom yes) (on_board yes)
@@
     (pin "2")
   )
+  (symbol (lib_id "iclr:292227-7") (at 259.08 25.4 0) (unit 1)
+    (in_bom yes) (on_board yes) (fields_autoplaced)
+    (property "Reference" "J5" (id 0) (at 273.05 31.75 0)
+      (effects (font (size 1.524 1.524)) (justify left))
+    )
+    (property "Value" "292227-7" (id 1) (at 273.05 35.56 0)
+      (effects (font (size 1.524 1.524)) (justify left))
+    )
+    (property "Footprint" "iclr:292227-7" (id 2) (at 269.24 34.544 0)
+      (effects (font (size 1.524 1.524)) hide)
+    )
+    (property "Datasheet" "" (id 3) (at 259.08 25.4 0)
+      (effects (font (size 1.524 1.524)))
+    )
+    (pin "1")
+    (pin "2")
+    (pin "3")
+    (pin "4")
+    (pin "5")
+    (pin "6")
+    (pin "7")
+  )
   (symbol (lib_id "Device:R_Small") (at 25.4 62.23 90) (unit 1)
     (in_bom yes) (on_board yes)
@@
     (pin "2")
   )
+  (symbol (lib_id "Connector:TestPoint") (at 20.32 137.16 90) (unit 1)
+    (in_bom yes) (on_board yes) (fields_autoplaced)
+    (property "Reference" "TP1" (id 0) (at 17.018 130.81 90))
+    (property "Value" "TestPoint" (id 1) (at 17.018 133.35 90))
+    (property "Footprint" "TestPoint:TestPoint_Pad_D1.0mm" (id 2) (at 20.32 132.08 0)
+      (effects (font (size 1.27 1.27)) hide)
+    )
+    (property "Datasheet" "~" (id 3) (at 20.32 132.08 0)
+      (effects (font (size 1.27 1.27)) hide)
+    )
+    (pin "1")
+  )
   (symbol (lib_id "power:+3.3V") (at 223.52 92.71 0) (unit 1)
     (in_bom yes) (on_board yes) (fields_autoplaced)
@@
       (effects (font (size 1.27 1.27)) (justify left))
     )
+    (pin "UC_Lipo_Scaled" output (at 59.69 33.02 0)
+      (effects (font (size 1.27 1.27)) (justify right))
+    )
   )
   (sheet (at 267.97 143.51) (size 13.97 11.43) (fields_autoplaced)
@@
       (reference "#PWR038") (unit 1) (value "GND") (footprint "")
     )
+    (path "/150d7a0e-7d8c-4788-bc30-4a3682bf4d09/3a502be0-672c-4774-a829-89ee66e4bf37"
+      (reference "#PWR039") (unit 1) (value "GND") (footprint "")
+    )
     (path "/ca0eab8e-e3fd-464d-bb03-d1603b8a651b/95fdd41f-879b-4183-897c-ad6f1e5df1b2"
       (reference "#PWR040") (unit 1) (value "+24V") (footprint "")
     )
+    (path "/698a410d-6a39-45b6-9e32-be9222181ad1/d2fc5bc4-3e53-4c7d-8982-f0c0392ae066"
+      (reference "#PWR041") (unit 1) (value "GND") (footprint "")
+    )
     (path "/ca0eab8e-e3fd-464d-bb03-d1603b8a651b/eec6d8e9-9bf8-4a69-a5ed-df68bef09560"
       (reference "#PWR042") (unit 1) (value "+24V") (footprint "")
@@
       (reference "#PWR0109") (unit 1) (value "+3.3V") (footprint "")
     )
-    (path "/698a410d-6a39-45b6-9e32-be9222181ad1/d99396c3-18e4-4d50-8cf6-3be3f26440a9"
-      (reference "#PWR0110") (unit 1) (value "VBUS") (footprint "")
-    )
     (path "/698a410d-6a39-45b6-9e32-be9222181ad1/f3ba7306-f05b-4d20-86ba-01c8bef6fcad"
       (reference "#PWR0111") (unit 1) (value "GND") (footprint "")
@@
       (reference "J4") (unit 1) (value "Micro_SD_Card_Det") (footprint "Connector_Card:microSD_HC_Hirose_DM3AT-SF-PEJM5")
     )
-    (path "/7b828807-61c4-4142-806c-aa288cdbf618"
-      (reference "J5") (unit 1) (value "Conn_01x07_Male") (footprint "Connector_JST:JST_GH_SM07B-GHS-TB_1x07-1MP_P1.25mm_Horizontal")
+    (path "/d33a8478-230a-43f7-abcf-13fc494c2482"
+      (reference "J5") (unit 1) (value "292227-7") (footprint "iclr:292227-7")
     )
     (path "/ca0eab8e-e3fd-464d-bb03-d1603b8a651b/a427a28b-3b40-4c8d-97e5-81714fd6f2be"
@@
       (reference "R22") (unit 1) (value "10k") (footprint "Resistor_SMD:R_0603_1608Metric")
     )
+    (path "/150d7a0e-7d8c-4788-bc30-4a3682bf4d09/3d8c465b-5d1a-4486-b744-787f839f7c0d"
+      (reference "R23") (unit 1) (value "7.5k") (footprint "Resistor_SMD:R_0603_1608Metric")
+    )
+    (path "/150d7a0e-7d8c-4788-bc30-4a3682bf4d09/b876f5bf-ac52-487e-8467-c3fea9a4dc29"
+      (reference "R24") (unit 1) (value "2.4k") (footprint "Resistor_SMD:R_0603_1608Metric")
+    )
     (path "/ca0eab8e-e3fd-464d-bb03-d1603b8a651b/24badbae-eef7-4d2c-a598-610e488ef81e"
       (reference "R25") (unit 1) (value "500") (footprint "Resistor_SMD:R_0603_1608Metric")
@@
       (reference "R27") (unit 1) (value "1K") (footprint "Resistor_SMD:R_0603_1608Metric")
     )
+    (path "/698a410d-6a39-45b6-9e32-be9222181ad1/10dddca5-8a78-4318-803f-5b3f3687bc7b"
+      (reference "R28") (unit 1) (value "24k") (footprint "Resistor_SMD:R_0603_1608Metric")
+    )
     (path "/ca0eab8e-e3fd-464d-bb03-d1603b8a651b/d7977444-08fa-4843-83fb-a1317f1a30c1"
       (reference "R29") (unit 1) (value "1K") (footprint "Resistor_SMD:R_0603_1608Metric")
     )
+    (path "/698a410d-6a39-45b6-9e32-be9222181ad1/ccc37dfa-7bf5-4bcb-94b8-dc78d821a9e6"
+      (reference "R30") (unit 1) (value "47k") (footprint "Resistor_SMD:R_0603_1608Metric")
+    )
     (path "/ca0eab8e-e3fd-464d-bb03-d1603b8a651b/c4d9bc73-27a3-45e8-9f5d-4537c1fd0ae5"
       (reference "R33") (unit 1) (value "500") (footprint "Resistor_SMD:R_0603_1608Metric")
@@
       (reference "R49") (unit 1) (value "60") (footprint "Resistor_SMD:R_0603_1608Metric")
     )
+    (path "/f0b7f9c2-6466-435c-88d0-33002b1d8435"
+      (reference "TP1") (unit 1) (value "TestPoint") (footprint "TestPoint:TestPoint_Pad_D1.0mm")
+    )
+    (path "/8cc63f8f-c92b-40c9-8c2b-aa1fa31e7980"
+      (reference "TP2") (unit 1) (value "TestPoint") (footprint "TestPoint:TestPoint_Pad_D1.0mm")
+    )
     (path "/c1ebf89d-7481-4930-9c04-a9a4c2a8bd4b"
       (reference "TP3") (unit 1) (value "TestPoint") (footprint "TestPoint:TestPoint_Pad_D1.0mm")
     )
-    (path "/9b4524df-73aa-42ff-b978-35806191ca38"
-      (reference "TP5") (unit 1) (value "TestPoint") (footprint "TestPoint:TestPoint_Pad_D1.0mm")
-    )
     (path "/ab8c7805-6159-4f04-8fa3-c39f9f102e96"
