File: PickleRick/usb_uart.kicad_sch (KiCad schematic)
At the start: 15 parts, among them J17 USB_C_Receptacle_USB2.0, U18 INTERFACE-CP2102-GMR(QFN28)

Commit message: first full layout of pickle complete
Parts:
- D21: footprint LED_SMD:LED_0603_1608Metric_Castellated -> LED_SMD:LED_0603_1608Metric
- TP30, TP31, TP32: footprint TestPoint:TestPoint_THTPad_1.0x1.0mm_Drill0.5mm -> TestPoint:TestPoint_Pad_D1.0mm
Changed lines of the file:
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@@
     (property "Reference" "D21" (id 0) (at 176.53 102.743 0))
     (property "Value" "USB_LED" (id 1) (at 176.53 105.0544 0))
-    (property "Footprint" "LED_SMD:LED_0603_1608Metric_Castellated" (id 2) (at 176.53 107.95 90)
+    (property "Footprint" "LED_SMD:LED_0603_1608Metric" (id 2) (at 176.53 107.95 90)
       (effects (font (size 1.27 1.27)) hide)
     )
@@
       (effects (font (size 1.27 1.27)) (justify left))
     )
-    (property "Footprint" "TestPoint:TestPoint_THTPad_1.0x1.0mm_Drill0.5mm" (id 2) (at 66.04 124.46 0)
+    (property "Footprint" "TestPoint:TestPoint_Pad_D1.0mm" (id 2) (at 66.04 124.46 0)
       (effects (font (size 1.27 1.27)) hide)
     )
@@
       (effects (font (size 1.27 1.27)) (justify left))
     )
-    (property "Footprint" "TestPoint:TestPoint_THTPad_1.0x1.0mm_Drill0.5mm" (id 2) (at 66.04 119.38 0)
+    (property "Footprint" "TestPoint:TestPoint_Pad_D1.0mm" (id 2) (at 66.04 119.38 0)
       (effects (font (size 1.27 1.27)) hide)
     )
@@
       (effects (font (size 1.27 1.27)) (justify left))
     )
-    (property "Footprint" "TestPoint:TestPoint_THTPad_1.0x1.0mm_Drill0.5mm" (id 2) (at 66.04 129.54 0)
-      (effects (font (size 1.27 1.27)) hide)
-    )
+    (property "Footprint" "TestPoint:TestPoint_Pad_D1.0mm" (id 2) (at 66.04 129.54 0)
+      (effects (font (size 1.27 1.27)) hide)
+    )

Commit message: pickle update
Parts:
- added R28: 24k, Resistor_SMD:R_0603_1608Metric, symbol Device:R_Small
- added R30: 47k, Resistor_SMD:R_0603_1608Metric, symbol Device:R_Small
Connections:
- net +3V3: now also C31.2, C33.2, U18.7 (REGIN)
- net GND: now also R30.1
- net VBUS: now also R28.2; no longer C31.2, C33.2, U18.7 (REGIN), U18.8 (VBUS)
- new net: R28.1, R30.2, U18.8 (VBUS)
Other:
- moved on the sheet: J17, R44, R45

Commit message: final changes to pick rick
Connections:
- net +3V3: now also C30.1; no longer C30.2
- net Data+: now also D20.3 (K); no longer D20.4 (K)
- net Data-: now also D20.4 (K); no longer D20.3 (K)
- net GND: now also C30.2; no longer C30.1
Other:
- moved on the sheet: C30
Changed lines of the file:
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@@
     (stroke (width 0) (type default) (color 0 0 0 0))
   )
-  (label "Data-" (at 146.05 149.86 90)
+  (label "Data-" (at 148.59 149.86 90)
     (effects (font (size 1.27 1.27)) (justify left bottom))
   )
@@
     (effects (font (size 1.27 1.27)) (justify left bottom))
   )
-  (label "Data+" (at 148.59 149.86 90)
+  (label "Data+" (at 146.05 149.86 90)
     (effects (font (size 1.27 1.27)) (justify left bottom))
   )
@@
     (pin "9")
   )
-  (symbol (lib_id "Device:CP1_Small") (at 111.76 63.5 0) (unit 1)
+  (symbol (lib_id "Device:CP1_Small") (at 111.76 63.5 180) (unit 1)
     (in_bom yes) (on_board yes)
-    (property "Reference" "C30" (id 0) (at 114.0714 62.3316 0)
+    (property "Reference" "C30" (id 0) (at 109.4486 64.6684 0)
       (effects (font (size 1.27 1.27)) (justify left))
     )
-    (property "Value" "4.7uF" (id 1) (at 114.0714 64.643 0)
+    (property "Value" "4.7uF" (id 1) (at 109.4486 62.357 0)
       (effects (font (size 1.27 1.27)) (justify left))
     )

Commit message: switched vspi and hspi labels so they are consistent with documentation
Parts:
- C30: footprint Capacitor_SMD:CP_Elec_3x5.3 -> Capacitor_SMD:C_0603_1608Metric; symbol Device:CP1_Small -> Device:C_Small
Changed lines of the file:
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@@
     (pin "9")
   )
-  (symbol (lib_id "Device:CP1_Small") (at 111.76 63.5 180) (unit 1)
+  (symbol (lib_id "Device:C_Small") (at 111.76 63.5 180) (unit 1)
     (in_bom yes) (on_board yes)
     (property "Reference" "C30" (id 0) (at 109.4486 64.6684 0)
@@
       (effects (font (size 1.27 1.27)) (justify left))
     )
-    (property "Footprint" "Capacitor_SMD:CP_Elec_3x5.3" (id 2) (at 111.76 63.5 0)
+    (property "Footprint" "Capacitor_SMD:C_0603_1608Metric" (id 2) (at 111.76 63.5 0)
       (effects (font (size 1.27 1.27)) hide)
     )
